Commit message: Add IMU sensor with plugin

File: models/bebop/urdf/multirotor_base.urdf.xacro (robot description, xacro)
@@ -39,10 +39,24 @@
         <origin xyz="0 0 0" rpy="0 0 0" />
       </inertial>
+    </link>
+    <gazebo reference="imu_link">
+      <gravity>true</gravity>
       <sensor name="imu_sensor" type="imu">
-        <pose>0 0 0 3.141593 0 0</pose>
-        <always_on>1</always_on>
-        <update_rate>1000.0</update_rate>
+        <always_on>true</always_on>
+        <update_rate>100</update_rate>
+        <visualize>true</visualize>
+        <topic>/bebop/imu</topic>
+        <plugin filename="libgazebo_ros_imu_sensor.so" name="imu_plugin">
+          <topicName>imu</topicName>
+          <bodyName>imu_link</bodyName>
+          <updateRateHZ>100.0</updateRateHZ>
+          <gaussianNoise>0.0</gaussianNoise>
+          <xyzOffset>0 0 0</xyzOffset>
+          <rpyOffset>0 0 0</rpyOffset>
+          <frameName>imu_link</frameName>
+        </plugin>
+        <pose>0 0 0 0 0 0</pose>
       </sensor>
-    </link>
+    </gazebo>
     <!-- IMU joint -->
     <joint name="imu_joint" type="revolute">

Commit message: Remove unneeded files

File: models/bebop/urdf/multirotor_base.urdf.xacro (robot description, xacro)
@@ -21,5 +21,5 @@
           <mesh filename="package://bebop_gazebo/meshes/${mesh_file}"
             scale="0.001 0.001 0.001" />
-          <!-- <box size="${body_width} ${body_width} ${body_height}"/> --> <!-- [m] [m] [m] -->
+          <!-- box size="${body_width} ${body_width} ${body_height}"/ --> <!-- [m] [m] [m] -->
         </geometry>
       </visual>

Commit message: Minor changes

File: models/bebop/urdf/multirotor_base.urdf.xacro (robot description, xacro)
@@ -232,5 +232,5 @@
         </geometry>
       </collision-->
-      <visual>
+      <!--visual>
         <origin xyz="0 0 0" rpy="0 0 0"/>
         <geometry>
@@ -238,5 +238,5 @@
         </geometry>
         <material name="red"/>
-      </visual>
+      </visual-->
       <inertial>
         <mass value="${camera_mass}" />
@@ -284,6 +284,6 @@
           <pointCloudTopicName>/${namespace}/camera/depth_registered/points</pointCloudTopicName>
           <frameName>camera</frameName>
-          <pointCloudCutoff>0.5</pointCloudCutoff>
-          <pointCloudCutoffMax>3.0</pointCloudCutoffMax>
+          <pointCloudCutoff>0.3</pointCloudCutoff>
+          <pointCloudCutoffMax>10.0</pointCloudCutoffMax>
           <distortionK1>0</distortionK1>
           <distortionK2>0</distortionK2>
