Commit message: Add kopterworx setup for SITL

File: models/bebop/urdf/bebop.urdf.xacro (robot description, xacro)
@@ -125,6 +125,6 @@
 	    <xacro:include filename="$(find velodyne_description)/urdf/VU-8.urdf.xacro"/>
 	    <VU-8 parent="base_link" name="leddar" topic="/leddar_points" hz="10" samples="440" gpu="false"
-	           min_range="0.5" >
-	        <origin xyz="0 0 0.05" rpy="0 0 0" />
+	           min_range="0.5" lasers="16">
+	        <origin xyz="0.1 0 0.15" rpy="3.141592653589793 0.1323284641020683 0." />
 	    </VU-8>
     </xacro:if>

Commit message: Change .dae mesh location

File: models/bebop/urdf/bebop.urdf.xacro (robot description, xacro)
@@ -125,5 +125,5 @@
 	    <xacro:include filename="$(find velodyne_description)/urdf/VU-8.urdf.xacro"/>
 	    <VU-8 parent="base_link" name="leddar" topic="/leddar_points" hz="10" samples="440" gpu="false"
-	           min_range="0.5" lasers="16">
+	           min_range="0.0" lasers="16">
 	        <origin xyz="0.1 0 0.15" rpy="3.141592653589793 0.1323284641020683 0." />
 	    </VU-8>

File: models/bebop/urdf/multirotor_base.urdf.xacro (robot description, xacro)
@@ -19,5 +19,5 @@
         <origin xyz="0 0 0" rpy="0 0 0" />
         <geometry>
-          <mesh filename="package://bebop_gazebo/meshes/${mesh_file}"
+          <mesh filename="package://ardupilot_gazebo/models/bebop/meshes/${mesh_file}"
             scale="0.001 0.001 0.001" />
           <!-- box size="${body_width} ${body_width} ${body_height}"/ --> <!-- [m] [m] [m] -->
@@ -98,5 +98,5 @@
         <geometry>
           <!-- <cylinder length="0.005" radius="${radius_rotor}"/> --> <!-- [m] -->
-          <mesh filename="package://bebop_gazebo/meshes/propeller_${direction}.dae"
+          <mesh filename="package://ardupilot_gazebo/models/bebop/meshes/propeller_${direction}.dae"
             scale="0.00055 0.00055 0.00055" />
           <!-- <box size="${2*radius_rotor} 0.01 0.005"/> -->

Commit message: Add paramters to ardupilot plugin

File: models/bebop/urdf/bebop.urdf.xacro (robot description, xacro)
@@ -72,5 +72,12 @@
 		<origin xyz="0.0 0.0 0.0" rpy="0.0 0.0 0.0" />
 	</xacro:odometry_plugin_macro>
-	<xacro:ardupilot>
+	<xacro:ardupilot
+		imu_topic="/bebop/imu"
+		control_topic="/gazebo/command/motor_speed"
+		imu_sensor_name="bebop::imu_link::imu_sensor"
+		rotor_0_joint="bebop::rotor_0_joint"
+		rotor_1_joint="bebop::rotor_1_joint"
+		rotor_2_joint="bebop::rotor_2_joint"
+		rotor_3_joint="bebop::rotor_3_joint">
 	</xacro:ardupilot>
     <link name="laser1D_link">

File: models/bebop/urdf/multirotor_base.urdf.xacro (robot description, xacro)
@@ -131,7 +131,10 @@
     </gazebo>
   </xacro:macro>
-  <xacro:macro name="ardupilot">
+  <xacro:macro name="ardupilot"
+    params="imu_topic control_topic imu_sensor_name rotor_0_joint rotor_1_joint rotor_2_joint rotor_3_joint">
      <gazebo>
         <plugin name="arducopter_plugin" filename="libArduPilotPlugin.so">
+        <imuTopicName>${imu_topic}</imuTopicName>
+        <controlTopicName>${control_topic}</controlTopicName>
         <fdm_addr>127.0.0.1</fdm_addr>
         <fdm_port_in>9002</fdm_port_in>
@@ -143,6 +146,7 @@
         <modelXYZToAirplaneXForwardZDown>0 0 0 3.141593 0 0</modelXYZToAirplaneXForwardZDown>
         <gazeboXYZToNED>0 0 0 3.141593 0 0</gazeboXYZToNED>
-        <imuName>bebop::imu_link::imu_sensor</imuName>
+        <imuName>${imu_sensor_name}</imuName>
         <connectionTimeoutMaxCount>5</connectionTimeoutMaxCount>
+        <!-- TODO: Remove this control parameters-->
         <control channel="0">
         <!--
@@ -162,5 +166,5 @@
           <cmd_max>3</cmd_max>
           <cmd_min>-3</cmd_min>
-          <jointName>bebop::rotor_1_joint</jointName>
+          <jointName>${rotor_1_joint}</jointName>
           <multiplier>600</multiplier>
           <controlVelocitySlowdownSim>1</controlVelocitySlowdownSim>
@@ -176,5 +180,5 @@
           <cmd_max>3</cmd_max>
           <cmd_min>-3</cmd_min>
-          <jointName>bebop::rotor_3_joint</jointName>
+          <jointName>${rotor_3_joint}</jointName>
           <multiplier>600</multiplier>
           <controlVelocitySlowdownSim>1</controlVelocitySlowdownSim>
@@ -190,5 +194,5 @@
           <cmd_max>3</cmd_max>
           <cmd_min>-3</cmd_min>
-          <jointName>bebop::rotor_0_joint</jointName>
+          <jointName>${rotor_0_joint}</jointName>
           <multiplier>-600</multiplier>
           <controlVelocitySlowdownSim>1</controlVelocitySlowdownSim>
@@ -204,5 +208,5 @@
           <cmd_max>3</cmd_max>
           <cmd_min>-3</cmd_min>
-          <jointName>bebop::rotor_2_joint</jointName>
+          <jointName>${rotor_2_joint}</jointName>
           <multiplier>-600</multiplier>
           <controlVelocitySlowdownSim>1</controlVelocitySlowdownSim>

Commit message: Add magnet to brick and bebop

File: models/bebop/urdf/bebop.urdf.xacro (robot description, xacro)
@@ -136,3 +136,38 @@
 	    </VU-8>
     </xacro:if>
+	<!--elektromagnet-->
+	<joint name="electromagnet_joint" type="fixed">
+		<axis xyz="0 1 0" />
+		<origin xyz="0.0 0.0 -0.075" rpy="0 0 0"/>
+		<parent link="base_link"/>
+		<child link="electromagnet_actuator"/>
+	</joint>
+	<link name="electromagnet_actuator">
+		<inertial>
+		<origin xyz="0 0 0" rpy="0 0 0" />
+		<mass value="0.025"/>
+		<inertia ixx="0.0001" ixy="0" ixz="0" iyy ="0.0001" iyz = "0" izz = "0.0001" />
+		</inertial>
+		<collision name="collision">
+		<geometry>
+			<cylinder radius="0.09" length="0.035"/>
+		</geometry>
+		</collision>
+		<visual>
+		<geometry>
+			<cylinder radius="0.09" length="0.035"/>
+		</geometry>
+		</visual>
+	</link>
+	<gazebo>
+		<plugin name="dipole_magnet" filename="libstorm_gazebo_dipole_magnet.so">
+			<bodyName>bebop::base_link</bodyName>
+			<dipole_moment>0 0 50</dipole_moment>
+			<!-- Set to false if not using ROS -->
+			<shouldPublish>true</shouldPublish>
+			<topicNs>magnet</topicNs>
+			<updateRate>100</updateRate>
+			<gain>1</gain>
+		</plugin>
+	</gazebo>
 </robot>

File: models/bebop/urdf/brick_red.urdf (robot description, URDF)
Before this commit: robot brick_green, 2 links, 1 joints
Links:
- link base_link: mass 1 -> 0.01
- link magnet_patch: geometry collision box size=0.1 0.025 0.0005; visual box size=0.2 0.125 0.001
Joints:
- joint patch_joint: origin xyz=0.0 0.0 0.101 rpy=0 0 0 -> xyz=0.0 0.0 0.1 rpy=0 0 0

Commit message: Add namespace for camera and change topic names to match RealSense

File: models/bebop/urdf/bebop.urdf.xacro (robot description, xacro)
@@ -151,10 +151,10 @@
 		<collision name="collision">
 		<geometry>
-			<cylinder radius="0.09" length="0.035"/>
+			<cylinder radius="0.08" length="0.035"/>
 		</geometry>
 		</collision>
 		<visual>
 		<geometry>
-			<cylinder radius="0.09" length="0.035"/>
+			<cylinder radius="0.08" length="0.035"/>
 		</geometry>
 		</visual>
@@ -166,5 +166,5 @@
 			<!-- Set to false if not using ROS -->
 			<shouldPublish>true</shouldPublish>
-			<topicNs>magnet</topicNs>
+			<topicNs>magnet_uav</topicNs>
 			<updateRate>100</updateRate>
 			<gain>1</gain>

File: models/bebop/urdf/bebop_base.urdf.xacro (robot description, xacro)
@@ -137,5 +137,5 @@
   <xacro:property name="camera_mass" value="1e-5"/>
   <xacro:cam
-    namespace="$(arg namespace)"
+    namespace="$(arg camera_namespace)"
     camera_link="${camera_link}"
     camera_mass="${camera_mass}"

File: models/bebop/urdf/multirotor_base.urdf.xacro (robot description, xacro)
@@ -279,9 +279,9 @@
           <updateRate>0.0</updateRate>
           <cameraName>camera_ir</cameraName>
-          <imageTopicName>/camera/color/image_raw</imageTopicName>
-          <cameraInfoTopicName>/camera/color/camera_info</cameraInfoTopicName>
+          <imageTopicName>/${namespace}/camera/color/image_raw</imageTopicName>
+          <cameraInfoTopicName>/${namespace}/camera/color/camera_info</cameraInfoTopicName>
           <depthImageTopicName>/camera/depth/image_raw</depthImageTopicName>
-          <depthImageCameraInfoTopicName>/camera/depth/camera_info</depthImageCameraInfoTopicName>
-          <pointCloudTopicName>/camera/depth/points</pointCloudTopicName>
+          <depthImageCameraInfoTopicName>/${namespace}/camera/depth/camera_info</depthImageCameraInfoTopicName>
+          <pointCloudTopicName>/${namespace}/camera/depth_registered/points</pointCloudTopicName>
           <frameName>camera</frameName>
           <pointCloudCutoff>0.5</pointCloudCutoff>

Commit message: Bebop camera setup - eagleblue

File: models/bebop/urdf/bebop.urdf.xacro (robot description, xacro)
@@ -151,5 +151,5 @@
 		<collision name="collision">
 		<geometry>
-			<cylinder radius="0.08" length="0.035"/>
+			<cylinder radius="0.04" length="0.035"/>
 		</geometry>
 		</collision>

File: models/bebop/urdf/bebop_base.urdf.xacro (robot description, xacro)
@@ -144,5 +144,5 @@
     <!--origin xyz="0.111 0 0.0217" rpy="0 1.57079632 0"/-->
     <!-- Side Facing Camera -->
-    <origin xyz="0 0.111 0.0217" rpy="-1.57079632 1.57079632 0"/>
+    <origin xyz="0 0.2 -0.3" rpy="-1.570796 1.570796 0"/>
     <xacro:insert_block name="camera_inertia"/>
   </xacro:cam>

File: models/bebop/urdf/multirotor_base.urdf.xacro (robot description, xacro)
@@ -232,5 +232,5 @@
         </geometry>
       </collision-->
-      <!--visual>
+      <visual>
         <origin xyz="0 0 0" rpy="0 0 0"/>
         <geometry>
@@ -238,8 +238,7 @@
         </geometry>
         <material name="red"/>
-      </visual-->
+      </visual>
       <inertial>
         <mass value="${camera_mass}" />
-        <origin xyz="0 0 0" rpy="0 0 0"/>
         <xacro:insert_block name="inertia"/>
       </inertial>

Commit message: Add flag for disabling velodyne and magnet

File: models/bebop/urdf/bebop.urdf.xacro (robot description, xacro)
@@ -2,4 +2,5 @@
 <robot name="bebop" xmlns:xacro="http://ros.org/wiki/xacro">
   <xacro:property name="enable_velodyne" value="$(arg enable_velodyne)"/>
+	<xacro:property name="enable_magnet" value="$(arg enable_magnet)"/>
   <xacro:property name="namespace" value="$(arg namespace)" />
   <xacro:property name="wind_force" value="$(arg wind_force)" />
@@ -137,4 +138,5 @@
     </xacro:if>
 	<!--elektromagnet-->
+	<xacro:if value="${enable_magnet}">
 	<joint name="electromagnet_joint" type="fixed">
 		<axis xyz="0 1 0" />
@@ -171,3 +173,4 @@
 		</plugin>
 	</gazebo>
+  </xacro:if>
 </robot>

Commit message: Remove wind arguments from bebop urdf

File: models/bebop/urdf/bebop.urdf.xacro (robot description, xacro)
@@ -4,10 +4,4 @@
 	<xacro:property name="enable_magnet" value="$(arg enable_magnet)"/>
   <xacro:property name="namespace" value="$(arg namespace)" />
-  <xacro:property name="wind_force" value="$(arg wind_force)" />
-  <xacro:property name="wind_start" value="$(arg wind_start)" />
-  <xacro:property name="wind_duration" value="$(arg wind_duration)" />
-  <xacro:property name="wind_direction_x" value="$(arg wind_direction_x)" />
-  <xacro:property name="wind_direction_y" value="$(arg wind_direction_y)" />
-  <xacro:property name="wind_direction_z" value="$(arg wind_direction_z)" />
   <!-- Instantiate bebop "mechanics" -->
 	<xacro:include filename="$(find ardupilot_gazebo)/models/bebop/urdf/bebop_base.urdf.xacro" />
