Commit message: Bebop with down-facing camera

File: models/bebop/urdf/bebop_base.urdf.xacro (robot description, xacro)
@@ -141,5 +141,5 @@
     camera_mass="${camera_mass}"
     parent="base_link">
-    <origin xyz="0.111 0 0.0217" rpy="0 0 0"/>
+    <origin xyz="0.111 0 0.0217" rpy="0 1.57079632 0"/>
     <xacro:insert_block name="camera_inertia"/>
   </xacro:cam>

Commit message: Add Side Facing Camera

File: models/bebop/urdf/bebop_base.urdf.xacro (robot description, xacro)
@@ -141,5 +141,8 @@
     camera_mass="${camera_mass}"
     parent="base_link">
-    <origin xyz="0.111 0 0.0217" rpy="0 1.57079632 0"/>
+    <!-- Front Facing Camera -->
+    <!--origin xyz="0.111 0 0.0217" rpy="0 1.57079632 0"/-->
+    <!-- Side Facing Camera -->
+    <origin xyz="0 0.111 0.0217" rpy="-1.57079632 1.57079632 0"/>
     <xacro:insert_block name="camera_inertia"/>
   </xacro:cam>

Commit message: Migrate common files to models/util folder.

File: models/bebop/urdf/bebop_base.urdf.xacro (robot description, xacro)
@@ -3,5 +3,6 @@
   <!-- Properties -->
   <xacro:property name="rotor_velocity_slowdown_sim" value="15" />
-  <xacro:property name="mesh_file" value="bebop.dae" />
+  <xacro:property name="mesh_file" value="ardupilot_gazebo/models/bebop/meshes/bebop.dae" />
+  <xacro:property name="mesh_scale" value="0.001" />
   <xacro:property name="mass" value="0.5" />  <!-- [kg] tum_sim 1.477 kg -->
   <xacro:property name="body_width" value="0.212" /> <!-- [m] old_value 0.1-->
@@ -36,5 +37,5 @@
   </xacro:property>
   <!-- Included URDF Files -->
-  <xacro:include filename="$(find ardupilot_gazebo)/models/bebop/urdf/multirotor_base.urdf.xacro" />
+  <xacro:include filename="$(find ardupilot_gazebo)/models/util/multirotor_base.urdf.xacro" />
   <!-- Instantiate multirotor_base_macro once -->
   <xacro:multirotor_base_macro
@@ -43,5 +44,7 @@
     body_width="${body_width}"
     body_height="${body_height}"
-    mesh_file="${mesh_file}">
+    mesh_file="${mesh_file}"
+    mesh_scale="${mesh_scale}">
+    <origin xyz="0 0 0" rpy="0 0 0"/>
     <xacro:insert_block name="body_inertia" />
   </xacro:multirotor_base_macro>

File: models/util/multirotor_base.urdf.xacro (robot description, xacro)
@@ -3,7 +3,8 @@
   <!-- Main multirotor link -->
   <xacro:macro name="multirotor_base_macro"
-    params="robot_namespace mass body_width body_height mesh_file *inertia">
+    params="robot_namespace mass body_width body_height mesh_file mesh_scale *origin *inertia">
     <link name="base_link"></link>
     <joint name="base_joint" type="fixed">
+      <xacro:insert_block name="origin"/>
       <origin xyz="0 0 0" rpy="0 0 0" />
       <parent link="base_link" />
@@ -19,6 +20,6 @@
         <origin xyz="0 0 0" rpy="0 0 0" />
         <geometry>
-          <mesh filename="package://ardupilot_gazebo/models/bebop/meshes/${mesh_file}"
-            scale="0.001 0.001 0.001" />
+          <mesh filename="package://${mesh_file}"
+            scale="${mesh_scale} ${mesh_scale} ${mesh_scale}" />
           <!-- box size="${body_width} ${body_width} ${body_height}"/ --> <!-- [m] [m] [m] -->
         </geometry>
@@ -27,5 +28,6 @@
         <origin xyz="0 0 0.0" rpy="0 0 0" />
         <geometry>
-          <box size="${body_width} ${body_width} ${body_height}" /> <!-- [m] [m] [m] -->
+          <mesh filename="package://${mesh_file}"
+            scale="${mesh_scale} ${mesh_scale} ${mesh_scale}" /> <!-- [m] [m] [m] -->
         </geometry>
       </collision>
@@ -45,10 +47,10 @@
         <update_rate>50</update_rate>
         <visualize>true</visualize>
-        <topic>/bebop/imu</topic>
+        <topic>/${robot_namespace}/imu</topic>
         <!-- IMU sensor has to be rotated accordint to the NED frame
              defined in the ArduPilot plugin -->
         <pose>0 0 0 3.141593 0 0</pose>
         <plugin filename="libgazebo_ros_imu_sensor.so" name="imu_plugin">
-          <topicName>/bebop/imu</topicName>
+          <topicName>/${robot_namespace}/imu</topicName>
           <bodyName>imu_link</bodyName>
           <updateRateHZ>50.0</updateRateHZ>
@@ -56,5 +58,5 @@
           <xyzOffset>0 0 0</xyzOffset>
           <rpyOffset>0 0 0</rpyOffset>
-          <frameName>bebop/imu</frameName>
+          <frameName>${robot_namespace}/imu</frameName>
         </plugin>
       </sensor>
@@ -70,5 +72,5 @@
     <gazebo>
       <plugin filename="librotors_gazebo_multirotor_base_plugin.so" name="rosbag">
-        <robotNamespace>$(arg namespace)</robotNamespace>
+        <robotNamespace>${robot_namespace}</robotNamespace>
         <linkName>base_link</linkName>
         <rotorVelocitySlowdownSim>${rotor_velocity_slowdown_sim}</rotorVelocitySlowdownSim>
@@ -98,5 +100,5 @@
         <geometry>
           <!-- <cylinder length="0.005" radius="${radius_rotor}"/> --> <!-- [m] -->
-          <mesh filename="package://ardupilot_gazebo/models/bebop/meshes/propeller_${direction}.dae"
+          <mesh filename="package://ardupilot_gazebo/models/util/propeller_${direction}.dae"
             scale="0.00055 0.00055 0.00055" />
           <!-- <box size="${2*radius_rotor} 0.01 0.005"/> -->

Commit message: [bebop_base.urdf] Add prop_scale parameter for vertical_rotor macros

File: models/bebop/urdf/bebop_base.urdf.xacro (robot description, xacro)
@@ -5,4 +5,5 @@
   <xacro:property name="mesh_file" value="ardupilot_gazebo/models/bebop/meshes/bebop.dae" />
   <xacro:property name="mesh_scale" value="0.001" />
+  <xacro:property name="prop_scale" value="0.00055" />
   <xacro:property name="mass" value="0.5" />  <!-- [kg] tum_sim 1.477 kg -->
   <xacro:property name="body_width" value="0.212" /> <!-- [m] old_value 0.1-->
@@ -65,5 +66,6 @@
     rotor_drag_coefficient="${rotor_drag_coefficient}"
     rolling_moment_coefficient="${rolling_moment_coefficient}"
-    color="Red">
+    color="Red"
+    prop_scale="${prop_scale}">
     <origin xyz="0.08440513 0.09784210 ${rotor_offset_top}" rpy="0 0 0" />
     <xacro:insert_block name="rotor_inertia" />
@@ -84,5 +86,6 @@
     rotor_drag_coefficient="${rotor_drag_coefficient}"
     rolling_moment_coefficient="${rolling_moment_coefficient}"
-    color="Blue">
+    color="Blue"
+    prop_scale="${prop_scale}">
     <origin xyz="0.08440513 -0.09784210 ${rotor_offset_top}" rpy="0 0 0" />
     <xacro:insert_block name="rotor_inertia" />
@@ -103,5 +106,6 @@
     rotor_drag_coefficient="${rotor_drag_coefficient}"
     rolling_moment_coefficient="${rolling_moment_coefficient}"
-    color="Blue">
+    color="Blue"
+    prop_scale="${prop_scale}">
     <origin xyz="-0.06853580 0.09784210 ${rotor_offset_top}" rpy="0 0 0" />
     <xacro:insert_block name="rotor_inertia" />
@@ -122,5 +126,6 @@
     rotor_drag_coefficient="${rotor_drag_coefficient}"
     rolling_moment_coefficient="${rolling_moment_coefficient}"
-    color="Red">
+    color="Red"
+    prop_scale="${prop_scale}">
     <origin xyz="-0.06853580 -0.09784210 ${rotor_offset_top}" rpy="0 0 0" />
     <xacro:insert_block name="rotor_inertia" />
