Commit message: Update properller offsets and properties.

File: models/kopterworx/urdf/kopterworx_base.urdf.xacro (robot description, xacro)
@@ -1,15 +1,21 @@
 <?xml version="1.0"?>
 <robot name="kopterworx" xmlns:xacro="http://ros.org/wiki/xacro">
+  <!-- Math constants -->
+  <xacro:property name="sin45" value="0.7071068" />
+  <xacro:property name="cos45" value="0.7071068" />
   <!-- Body Properties -->
   <xacro:property name="rotor_velocity_slowdown_sim" value="15" />
-  <xacro:property name="mesh_file" value="ardupilot_gazebo/models/kopterworx/meshes/kopterworx_model.stl" />
+  <xacro:property name="mesh_file" value="ardupilot_gazebo/models/kopterworx/meshes/kopterworx_model_simple.dae" />
   <xacro:property name="mesh_scale" value="0.1" />
+  <xacro:property name="prop_scale" value="0.002" />
   <xacro:property name="mass" value="9" />  <!-- [kg] -->
   <xacro:property name="body_width" value="0.3" /> <!-- [m] -->
-  <xacro:property name="body_height" value="0.3" /> <!-- [m] -->
-  <xacro:property name="arm_length" value="0.12905" /> <!-- [m] -->
+  <xacro:property name="body_height" value="0.6" /> <!-- [m] -->
+  <xacro:property name="arm_length" value="0.52" /> <!-- [m] -->
+  <xacro:property name="rotor_x_offset" value="${arm_length*cos45}" /> <!-- [m] -->
+  <xacro:property name="rotor_y_offset" value="${arm_length*sin45}" /> <!-- [m] -->
+  <xacro:property name="rotor_offset_top" value="0.115" /> <!-- [m] -->
   <!-- Rotor constants -->
-  <xacro:property name="mass_rotor" value="0.375" /> <!-- [kg] -->
-  <xacro:property name="rotor_offset_top" value="0.03" /> <!-- [m] -->
+  <xacro:property name="mass_rotor" value="0.01" /> <!-- [kg] -->
   <xacro:property name="radius_rotor" value="0.285" /> <!-- [m] -->
   <xacro:property name="motor_constant" value="8.54858e-06" /> <!-- [kg*m/s^2] -->
@@ -20,7 +26,4 @@
   <xacro:property name="rotor_drag_coefficient" value="8.06428e-05" />
   <xacro:property name="rolling_moment_coefficient" value="0.000001" />
-  <!-- Math constants -->
-  <xacro:property name="sin45" value="0.7071068" />
-  <xacro:property name="cos45" value="0.7071068" />
   <!-- Property Blocks -->
   <xacro:property name="body_inertia">
@@ -60,6 +63,7 @@
     rotor_drag_coefficient="${rotor_drag_coefficient}"
     rolling_moment_coefficient="${rolling_moment_coefficient}"
-    color="Red">
-    <origin xyz="0.08440513 0.09784210 ${rotor_offset_top}" rpy="0 0 0" />
+    color="Red"
+    prop_scale="${prop_scale}">
+    <origin xyz="${rotor_x_offset} ${rotor_y_offset} ${rotor_offset_top}" rpy="0 0 0" />
     <xacro:insert_block name="rotor_inertia" />
   </xacro:vertical_rotor>
@@ -79,6 +83,7 @@
     rotor_drag_coefficient="${rotor_drag_coefficient}"
     rolling_moment_coefficient="${rolling_moment_coefficient}"
-    color="Blue">
-    <origin xyz="0.08440513 -0.09784210 ${rotor_offset_top}" rpy="0 0 0" />
+    color="Blue"
+    prop_scale="${prop_scale}">
+    <origin xyz="${rotor_x_offset} -${rotor_y_offset} ${rotor_offset_top}" rpy="0 0 0" />
     <xacro:insert_block name="rotor_inertia" />
   </xacro:vertical_rotor>
@@ -98,6 +103,7 @@
     rotor_drag_coefficient="${rotor_drag_coefficient}"
     rolling_moment_coefficient="${rolling_moment_coefficient}"
-    color="Blue">
-    <origin xyz="-0.06853580 0.09784210 ${rotor_offset_top}" rpy="0 0 0" />
+    color="Blue"
+    prop_scale="${prop_scale}">
+    <origin xyz="-${rotor_x_offset} ${rotor_y_offset} ${rotor_offset_top}" rpy="0 0 0" />
     <xacro:insert_block name="rotor_inertia" />
   </xacro:vertical_rotor>
@@ -117,6 +123,7 @@
     rotor_drag_coefficient="${rotor_drag_coefficient}"
     rolling_moment_coefficient="${rolling_moment_coefficient}"
-    color="Red">
-    <origin xyz="-0.06853580 -0.09784210 ${rotor_offset_top}" rpy="0 0 0" />
+    color="Red"
+    prop_scale="${prop_scale}">
+    <origin xyz="-${rotor_x_offset} -${rotor_y_offset} ${rotor_offset_top}" rpy="0 0 0" />
     <xacro:insert_block name="rotor_inertia" />
   </xacro:vertical_rotor>

Commit message: Adjust kopterworx body inertia and motor constants.

File: models/kopterworx/urdf/kopterworx_base.urdf.xacro (robot description, xacro)
@@ -19,6 +19,6 @@
   <xacro:property name="mass_rotor" value="0.01" /> <!-- [kg] -->
   <xacro:property name="radius_rotor" value="0.285" /> <!-- [m] -->
-  <xacro:property name="motor_constant" value="0.00024407246" /> <!-- [kg*m/s^2] -->
-  <xacro:property name="moment_constant" value="0.016" /> <!-- [m] -->
+  <xacro:property name="motor_constant" value="0.000285576174524687" /> <!-- [kg*m/s^2] -->
+  <xacro:property name="moment_constant" value="0.041365783102071" /> <!-- [m] -->
   <xacro:property name="time_constant_up" value="0.0125" /> <!-- [s] -->
   <xacro:property name="time_constant_down" value="0.0125" /> <!-- [s] -->
@@ -28,5 +28,5 @@
   <!-- Property Blocks -->
   <xacro:property name="body_inertia">
-    <inertia ixx="0.274253" ixy="0.0" ixz="0.0" iyy="0.274253" iyz="0.0" izz="0.469118" />
+    <inertia ixx="0.303755" ixy="0.0004484919" ixz="0.0010159727" iyy="0.27722" iyz="-0.001806885" izz="0.469164" />
   </xacro:property>
   <!-- inertia of a single rotor, assuming it is a cuboid. Height=3mm, width=15mm -->
