Commit message: Added tilt-rotors and movable mass to urdf

File: models/kopterworx/urdf/kopterworx_tilt.urdf.xacro (robot description, xacro)
@@ -3,37 +3,38 @@
   <xacro:property name="namespace" value="$(arg namespace)" />
   <xacro:property name="enable_velodyne" value="$(arg enable_velodyne)"/>
-	<xacro:property name="enable_rotating_velodyne" value="$(arg enable_rotating_velodyne)" />
-	<xacro:property name="fdm_port_in" value="$(arg fdm_port_in)"/>
-	<xacro:property name="fdm_port_out" value="$(arg fdm_port_out)"/>
-	<xacro:property name="max_range" value="$(arg max_range)"/>
-	<gazebo>
-    <plugin name="gazebo_ros_control" filename="libgazebo_ros_control.so">
-      <robotNamespace>/$(arg namespace)</robotNamespace>
-      <robotParam>/$(arg namespace)/robot_description </robotParam>
-      <robotSimType>gazebo_ros_control/DefaultRobotHWSim</robotSimType>
-    </plugin>
+  <xacro:property name="enable_magnet" value="$(arg enable_magnet)"/>
+  <xacro:property name="enable_rotating_velodyne" value="$(arg enable_rotating_velodyne)" />
+  <xacro:property name="fdm_port_in" value="$(arg fdm_port_in)"/>
+  <xacro:property name="fdm_port_out" value="$(arg fdm_port_out)"/>
+  <xacro:property name="max_range" value="$(arg max_range)"/>
+  <xacro:property name="laser_count" value="$(arg laser_count)"/>
+  <gazebo>
+  	<plugin name="gazebo_ros_control" filename="libgazebo_ros_control.so">
+    	<robotNamespace>/$(arg namespace)</robotNamespace>
+    	<robotParam>/$(arg namespace)/robot_description </robotParam>
+    	<robotSimType>gazebo_ros_control/DefaultRobotHWSim</robotSimType>
+  	</plugin>
   </gazebo>
-	<xacro:property name="horizontal_velodyne_origin">
-    <origin xyz="0.08 0. -0.1578" rpy="-3.141592653589793 0.1323284641020683 0." />
-	</xacro:property>
-	<xacro:property name="front_facing_camera">
-		<origin xyz="0.2 0 0.05" rpy="0 0 0"/>
-	</xacro:property>
-	<xacro:property name="down_facing_camera">
-	  <origin xyz="0 0.2 -0.3" rpy="-1.570796 1.570796 0"/>
-	</xacro:property>
+  <xacro:property name="horizontal_velodyne_origin">
+	<origin xyz="0.08 0. -0.1578" rpy="-3.141592653589793 0.1323284641020683 0." />
+  </xacro:property>
+  <xacro:property name="front_facing_camera">
+	<origin xyz="0.2 0 0.05" rpy="0 0 0"/>
+  </xacro:property>
+  <xacro:property name="down_facing_camera">
+    <origin xyz="0 0.2 -0.3" rpy="-1.570796 1.570796 0"/>
+  </xacro:property>
   <xacro:property name="camera_mass" value="1e-5"/>
-	<xacro:property name="camera_size" value="0.05" />
+  <xacro:property name="camera_size" value="0.05" />
   <xacro:property name="camera_inertia">
-    <inertia
-    ixx="1e-12"
-    iyy="1e-12"
-    izz="1e-12"
-    ixy="0.0" ixz="0.0" iyz="0.0" />
+    <inertia ixx="1e-12" iyy="1e-12" izz="1e-12" ixy="0.0" ixz="0.0" iyz="0.0" />
   </xacro:property>
   <!-- Instantiate kopterworx mechanics "mechanics" -->
-	<xacro:include filename="$(find ardupilot_gazebo)/models/kopterworx/urdf/kopterworx_base.urdf.xacro" />
+  <xacro:include filename="$(find ardupilot_gazebo)/models/kopterworx/urdf/kopterworx_tilt_base.urdf.xacro" />
   <xacro:include filename="$(find rotors_description)/urdf/component_snippets.xacro" />
-	<!-- Ardupilot plugin -->
+  <!-- Ardupilot plugin
+    NOTE: thrust_multiplier
+      Value is tuned in order for mavros/setpoint_raw/attitude/thrust to reflect real-world behavior.
+  -->
   <xacro:ardupilot
 		imu_topic="/${namespace}/imu"
@@ -48,4 +49,16 @@
 		fdm_port_out="${fdm_port_out}">
 	</xacro:ardupilot>
+  <xacro:if value="${enable_magnet}">
+    <xacro:magnet_plugin
+      parent="${namespace}/base_link_inertia"
+      namespace="${namespace}"
+      name="uav_magnet"
+      moment_x="0"
+      moment_y="0"
+      moment_z="50"
+      length="0.25"
+      offset="0.07">
+    </xacro:magnet_plugin>
+  </xacro:if>
 	<xacro:if value="${enable_velodyne}">
 		<xacro:if value="${enable_rotating_velodyne}">
@@ -60,5 +73,5 @@
 				min_range="1"
 				max_range="${max_range}"
-				lasers="16">
+				lasers="32">
 				<xacro:insert_block name="horizontal_velodyne_origin"/>
 			</xacro:lidar-x>
@@ -75,5 +88,5 @@
 				min_range="1"
 				max_range="${max_range}"
-				lasers="16">
+				lasers="32">
 				<xacro:insert_block name="horizontal_velodyne_origin"/>
 			</xacro:lidar-x>

File: models/kopterworx/urdf/kopterworx_tilt_base.urdf.xacro (robot description, xacro)
@@ -26,4 +26,12 @@
   <xacro:property name="rotor_drag_coefficient" value="8.06428e-05" />
   <xacro:property name="rolling_moment_coefficient" value="0.000001" />
+  <!-- Tilt link constants -->
+  <xacro:property name="tilt_mass" value="0.1" />
+  <xacro:property name="tilt_length" value="0.05" />
+  <xacro:property name="tilt_radius" value="0.005" />
+  <xacro:property name="tilt_x_offset" value="${arm_length*cos45 + 0.0065}" />
+  <xacro:property name="tilt_y_offset" value="${arm_length*sin45 + 0.0065}" />
+  <xacro:property name="tilt_z_offset" value="0.1" />
+  <xacro:property name="prop_z_offset" value="${tilt_length}" />
   <!-- Property Blocks -->
   <xacro:property name="body_inertia">
@@ -36,4 +44,5 @@
   <!-- Included URDF Files -->
   <xacro:include filename="$(find ardupilot_gazebo)/models/util/multirotor_base.urdf.xacro" />
+  <xacro:include filename="$(find ardupilot_gazebo)/models/util/multirotor_tilt.urdf.xacro" />
   <!-- Instantiate multirotor_base_macro once -->
   <xacro:multirotor_base_macro
@@ -47,4 +56,66 @@
     <xacro:insert_block name="body_inertia" />
   </xacro:multirotor_base_macro>
+  <!-- Instantiate tilt-links -->
+  <xacro:prop_tilt
+    robot_namespace="$(arg namespace)"
+    parent="$(arg namespace)/base_link"
+    number="1"
+    x_axis="0.7071068"
+    y_axis="-0.7071068"
+    mass="${tilt_mass}"
+    length="${tilt_length}"
+    radius="${tilt_radius}">
+    <origin xyz="${tilt_x_offset} ${tilt_y_offset} ${tilt_z_offset}" rpy="0 0 0" />
+  </xacro:prop_tilt>
+  <xacro:prop_tilt
+    robot_namespace="$(arg namespace)"
+    parent="$(arg namespace)/base_link"
+    number="0"
+    x_axis="0.7071068"
+    y_axis="0.7071068"
+    mass="${tilt_mass}"
+    length="${tilt_length}"
+    radius="${tilt_radius}">
+    <origin xyz="${tilt_x_offset} -${tilt_y_offset} ${tilt_z_offset}" rpy="0 0 0" />
+  </xacro:prop_tilt>
+  <xacro:prop_tilt
+    robot_namespace="$(arg namespace)"
+    parent="$(arg namespace)/base_link"
+    number="2"
+    x_axis="0.7071068"
+    y_axis="0.7071068"
+    mass="${tilt_mass}"
+    length="${tilt_length}"
+    radius="${tilt_radius}">
+    <origin xyz="-${tilt_x_offset} ${tilt_y_offset} ${tilt_z_offset}" rpy="0 0 0" />
+  </xacro:prop_tilt>
+  <xacro:prop_tilt
+    robot_namespace="$(arg namespace)"
+    parent="$(arg namespace)/base_link"
+    number="3"
+    x_axis="0.7071068"
+    y_axis="-0.7071068"
+    mass="${tilt_mass}"
+    length="${tilt_length}"
+    radius="${tilt_radius}">
+    <origin xyz="-${tilt_x_offset} -${tilt_y_offset} ${tilt_z_offset}" rpy="0 0 0" />
+  </xacro:prop_tilt>
+  <!-- Instantiate tilt-joint transmissions -->
+  <xacro:tilt_joint_transmission
+    number="1"
+    joint_name="red/tilt_joint_1">
+  </xacro:tilt_joint_transmission>
+  <xacro:tilt_joint_transmission
+    number="0"
+    joint_name="red/tilt_joint_0">
+  </xacro:tilt_joint_transmission>
+  <xacro:tilt_joint_transmission
+    number="2"
+    joint_name="red/tilt_joint_2">
+  </xacro:tilt_joint_transmission>
+  <xacro:tilt_joint_transmission
+    number="3"
+    joint_name="red/tilt_joint_3">
+  </xacro:tilt_joint_transmission>
   <!-- Instantiate rotors -->
   <xacro:vertical_rotor
@@ -54,5 +125,5 @@
     motor_constant="${motor_constant}"
     moment_constant="${moment_constant}"
-    parent="$(arg namespace)/base_link"
+    parent="$(arg namespace)/tilt_link_1"
     mass_rotor="${mass_rotor}"
     radius_rotor="${radius_rotor}"
@@ -65,5 +136,5 @@
     color="Red"
     prop_scale="${prop_scale}">
-    <origin xyz="${rotor_x_offset} ${rotor_y_offset} ${rotor_offset_top}" rpy="0 0 0" />
+    <origin xyz="0 0 ${prop_z_offset}" rpy="0 0 0" />
     <xacro:insert_block name="rotor_inertia" />
   </xacro:vertical_rotor>
@@ -74,5 +145,5 @@
     motor_constant="${motor_constant}"
     moment_constant="${moment_constant}"
-    parent="$(arg namespace)/base_link"
+    parent="$(arg namespace)/tilt_link_0"
     mass_rotor="${mass_rotor}"
     radius_rotor="${radius_rotor}"
@@ -85,5 +156,5 @@
     color="Blue"
     prop_scale="${prop_scale}">
-    <origin xyz="${rotor_x_offset} -${rotor_y_offset} ${rotor_offset_top}" rpy="0 0 0" />
+    <origin xyz="0 0 ${prop_z_offset}" rpy="0 0 0" />
     <xacro:insert_block name="rotor_inertia" />
   </xacro:vertical_rotor>
@@ -94,5 +165,5 @@
     motor_constant="${motor_constant}"
     moment_constant="${moment_constant}"
-    parent="$(arg namespace)/base_link"
+    parent="$(arg namespace)/tilt_link_2"
     mass_rotor="${mass_rotor}"
     radius_rotor="${radius_rotor}"
@@ -105,5 +176,5 @@
     color="Blue"
     prop_scale="${prop_scale}">
-    <origin xyz="-${rotor_x_offset} ${rotor_y_offset} ${rotor_offset_top}" rpy="0 0 0" />
+    <origin xyz="0 0 ${prop_z_offset}" rpy="0 0 0" />
     <xacro:insert_block name="rotor_inertia" />
   </xacro:vertical_rotor>
@@ -114,5 +185,5 @@
     motor_constant="${motor_constant}"
     moment_constant="${moment_constant}"
-    parent="$(arg namespace)/base_link"
+    parent="$(arg namespace)/tilt_link_3"
     mass_rotor="${mass_rotor}"
     radius_rotor="${radius_rotor}"
@@ -125,7 +196,26 @@
     color="Red"
     prop_scale="${prop_scale}">
-    <origin xyz="-${rotor_x_offset} -${rotor_y_offset} ${rotor_offset_top}" rpy="0 0 0" />
-    <xacro:insert_block name="rotor_inertia" />
-  </xacro:vertical_rotor>
+    <origin xyz="0 0 ${prop_z_offset}" rpy="0 0 0" />
+    <xacro:insert_block name="rotor_inertia" />
+  </xacro:vertical_rotor>
+  <!-- Instantiate movable mass -->
+  <xacro:movable_mass_linear
+    robot_namespace="$(arg namespace)"
+    number="0"
+    parent="$(arg namespace)/base_link"
+    mass="0.5"
+    radius="0.05"
+    path_len="1"
+    color="Yellow"
+    x_axis="1"
+    y_axis="0"
+    z_axis="0">
+    <origin xyz="0 0 -0.15" rpy="0 0 0" />
+  </xacro:movable_mass_linear>
+  <!-- Instantiate movable mass transmission -->
+  <xacro:movable_mass_transmission
+    number="0"
+    joint_name="red/movable_mass_joint_0">
+  </xacro:movable_mass_transmission>
   <gazebo reference="$(arg namespace)/base_link">
     <dampingFactor>0.001</dampingFactor>

File: models/util/multirotor_base.urdf.xacro (robot description, xacro)
@@ -32,6 +32,5 @@
       <visual>
         <geometry>
-          <mesh filename="package://${mesh_file}"
-            scale="${mesh_scale} ${mesh_scale} ${mesh_scale}" />
+          <mesh filename="package://${mesh_file}" scale="${mesh_scale} ${mesh_scale} ${mesh_scale}" />
           <!--box size="${body_width} ${body_width} ${body_height}"/--> <!-- [m] [m] [m] -->
         </geometry>
@@ -48,6 +47,5 @@
     <link name="imu_link">
       <inertial>
-        <inertia ixx="0.001" ixy="0.0" ixz="0.0" iyy="0.001" iyz="0.0"
-          izz="0.001" />
+        <inertia ixx="0.001" ixy="0.0" ixz="0.0" iyy="0.001" iyz="0.0" izz="0.001" />
         <mass value="0.01" />  <!-- [kg] -->
         <origin xyz="0 0 0" rpy="0 0 0" />
@@ -102,5 +100,5 @@
     <!-- TODO(ff): not currently set because it's not yet supported -->
     <!-- <gazebo reference="rotor_${motor_number}_joint"> <axis> <xyz>0 0 1</xyz>
-      <limit> <velocity> ${max_rot_velocity} </velocity> </limit> </axis> </gazebo> -->
+    <limit> <velocity> ${max_rot_velocity} </velocity> </limit> </axis> </gazebo> -->
     <link name="${robot_namespace}/rotor_${motor_number}">
       <inertial>
