Commit message: Added movable masses for manipulator moment cancelation

File: models/kopterworx/urdf/kopterworx_tilt_base.urdf.xacro (robot description, xacro)
@@ -199,5 +199,5 @@
     <xacro:insert_block name="rotor_inertia" />
   </xacro:vertical_rotor>
-  <!-- Instantiate movable mass -->
+  <!-- Instantiate manipulator center of mass -->
   <xacro:movable_mass_linear
     robot_namespace="$(arg namespace)"
@@ -206,5 +206,6 @@
     mass="0.5"
     radius="0.05"
-    path_len="1"
+    limit_low="-0.2"
+    limit_high="0.2"
     color="Yellow"
     x_axis="1"
@@ -213,9 +214,83 @@
     <origin xyz="0 0 -0.15" rpy="0 0 0" />
   </xacro:movable_mass_linear>
-  <!-- Instantiate movable mass transmission -->
-  <xacro:movable_mass_transmission
+  <!-- Instantiate manipulator center of mass transmission -->
+  <xacro:movable_mass_pos_transmission
     number="0"
     joint_name="red/movable_mass_joint_0">
-  </xacro:movable_mass_transmission>
+  </xacro:movable_mass_pos_transmission>
+  <!-- Instantiate movable masses -->
+  <xacro:movable_mass_linear
+    robot_namespace="$(arg namespace)"
+    number="1"
+    parent="$(arg namespace)/base_link"
+    mass="0.25"
+    radius="0.03"
+    limit_low="0.2"
+    limit_high="0.5"
+    color="Orange"
+    x_axis="${sin45}"
+    y_axis="${-sin45}"
+    z_axis="0">
+    <origin xyz="0 0 0" rpy="0 0 0" />
+  </xacro:movable_mass_linear>
+  <xacro:movable_mass_linear
+    robot_namespace="$(arg namespace)"
+    number="2"
+    parent="$(arg namespace)/base_link"
+    mass="0.25"
+    radius="0.03"
+    limit_low="0.2"
+    limit_high="0.5"
+    color="Orange"
+    x_axis="${sin45}"
+    y_axis="${sin45}"
+    z_axis="0">
+    <origin xyz="0 0 0" rpy="0 0 0" />
+  </xacro:movable_mass_linear>
+  <xacro:movable_mass_linear
+    robot_namespace="$(arg namespace)"
+    number="3"
+    parent="$(arg namespace)/base_link"
+    mass="0.25"
+    radius="0.03"
+    limit_low="0.2"
+    limit_high="0.5"
+    color="Orange"
+    x_axis="${-sin45}"
+    y_axis="${sin45}"
+    z_axis="0">
+    <origin xyz="0 0 0" rpy="0 0 0" />
+  </xacro:movable_mass_linear>
+  <xacro:movable_mass_linear
+    robot_namespace="$(arg namespace)"
+    number="4"
+    parent="$(arg namespace)/base_link"
+    mass="0.25"
+    radius="0.03"
+    limit_low="0.2"
+    limit_high="0.5"
+    color="Orange"
+    x_axis="${-sin45}"
+    y_axis="${-sin45}"
+    z_axis="0">
+    <origin xyz="0 0 0" rpy="0 0 0" />
+  </xacro:movable_mass_linear>
+  <!-- Instantiate movable masses transmissions -->
+  <xacro:movable_mass_vel_transmission
+    number="1"
+    joint_name="red/movable_mass_joint_1">
+  </xacro:movable_mass_vel_transmission>
+  <xacro:movable_mass_vel_transmission
+    number="2"
+    joint_name="red/movable_mass_joint_2">
+  </xacro:movable_mass_vel_transmission>
+  <xacro:movable_mass_vel_transmission
+    number="3"
+    joint_name="red/movable_mass_joint_3">
+  </xacro:movable_mass_vel_transmission>
+  <xacro:movable_mass_vel_transmission
+    number="4"
+    joint_name="red/movable_mass_joint_4">
+  </xacro:movable_mass_vel_transmission>
   <gazebo reference="$(arg namespace)/base_link">
     <dampingFactor>0.001</dampingFactor>

File: models/util/multirotor_tilt.urdf.xacro (robot description, xacro)
@@ -30,5 +30,5 @@
   <!-- Macro for movable mass on a straight line. -->
   <xacro:macro name="movable_mass_linear"
-    params="robot_namespace number parent mass radius path_len color x_axis y_axis z_axis *origin">
+    params="robot_namespace number parent mass radius limit_low limit_high color x_axis y_axis z_axis *origin">
     <joint name="${robot_namespace}/movable_mass_joint_${number}" type="prismatic">
       <xacro:insert_block name="origin"/>
@@ -36,5 +36,5 @@
       <parent link="${parent}"/>
       <child link="${robot_namespace}/movable_mass_link_${number}"/>
-      <limit lower="${-path_len/2}" upper="${path_len/2}" effort="10000" velocity="20"/>
+      <limit lower="${limit_low}" upper="${limit_high}" effort="10000" velocity="20"/>
     </joint>
     <link name="${robot_namespace}/movable_mass_link_${number}">
@@ -70,6 +70,6 @@
     </transmission>
   </xacro:macro>
-  <xacro:macro name="movable_mass_transmission" params="number joint_name">
-    <transmission name="movable_mass_transmission_${number}">
+  <xacro:macro name="movable_mass_pos_transmission" params="number joint_name">
+    <transmission name="movable_mass_pos_transmission_${number}">
       <type>transmission_interface/SimpleTransmission</type>
       <actuator name="movable_mass_motor_${number}">
@@ -81,3 +81,14 @@
     </transmission>
   </xacro:macro>
+  <xacro:macro name="movable_mass_vel_transmission" params="number joint_name">
+    <transmission name="movable_mass_vel_transmission_${number}">
+      <type>transmission_interface/SimpleTransmission</type>
+      <actuator name="movable_mass_motor_${number}">
+        <mechanicalReduction>1</mechanicalReduction>
+      </actuator>
+      <joint name="${joint_name}">
+        <hardwareInterface>hardware_interface/VelocityJointInterface</hardwareInterface>
+      </joint>
+    </transmission>
+  </xacro:macro>
 </robot>
