Commit message: Kopterworx SITL - rotor propery adjustment.

File: models/kopterworx/urdf/kopterworx.urdf.xacro (robot description, xacro)
@@ -5,3 +5,13 @@
 	<xacro:include filename="$(find ardupilot_gazebo)/models/kopterworx/urdf/kopterworx_base.urdf.xacro" />
   <xacro:include filename="$(find rotors_description)/urdf/component_snippets.xacro" />
+  	<xacro:ardupilot
+		imu_topic="/kopterworx/imu"
+		control_topic="/gazebo/command/motor_speed"
+		imu_sensor_name="kopterworx::imu_link::imu_sensor"
+		rotor_0_joint="kopterworx::rotor_0_joint"
+		rotor_1_joint="kopterworx::rotor_1_joint"
+		rotor_2_joint="kopterworx::rotor_2_joint"
+		rotor_3_joint="kopterworx::rotor_3_joint"
+		thrust_multiplier="600">
+	</xacro:ardupilot>
 </robot>

File: models/kopterworx/urdf/kopterworx_base.urdf.xacro (robot description, xacro)
@@ -19,14 +19,14 @@
   <xacro:property name="mass_rotor" value="0.01" /> <!-- [kg] -->
   <xacro:property name="radius_rotor" value="0.285" /> <!-- [m] -->
-  <xacro:property name="motor_constant" value="8.54858e-06" /> <!-- [kg*m/s^2] -->
+  <xacro:property name="motor_constant" value="0.00024407246" /> <!-- [kg*m/s^2] -->
   <xacro:property name="moment_constant" value="0.016" /> <!-- [m] -->
   <xacro:property name="time_constant_up" value="0.0125" /> <!-- [s] -->
   <xacro:property name="time_constant_down" value="0.0125" /> <!-- [s] -->
-  <xacro:property name="max_rot_velocity" value="1475" /> <!-- [rad/s] -->
+  <xacro:property name="max_rot_velocity" value="600" /> <!-- [rad/s] -->
   <xacro:property name="rotor_drag_coefficient" value="8.06428e-05" />
   <xacro:property name="rolling_moment_coefficient" value="0.000001" />
   <!-- Property Blocks -->
   <xacro:property name="body_inertia">
-    <inertia ixx="0.00389" ixy="0.0" ixz="0.0" iyy="0.00389" iyz="0.0" izz="0.0078" />
+    <inertia ixx="0.274253" ixy="0.0" ixz="0.0" iyy="0.274253" iyz="0.0" izz="0.469118" />
   </xacro:property>
   <!-- inertia of a single rotor, assuming it is a cuboid. Height=3mm, width=15mm -->

Commit message: [kopterworx] Add velodyne to kopterworx.

File: models/kopterworx/urdf/kopterworx.urdf.xacro (robot description, xacro)
@@ -2,8 +2,13 @@
 <robot name="kopterworx" xmlns:xacro="http://ros.org/wiki/xacro">
   <xacro:property name="namespace" value="$(arg namespace)" />
-  <!-- Instantiate bebop "mechanics" -->
+  <xacro:property name="enable_velodyne" value="$(arg enable_velodyne)"/>
+	<xacro:property name="horizontal_velodyne_origin">
+    <origin xyz="0.08 0. -0.1578" rpy="3.141592653589793 0.1323284641020683 0." />
+	</xacro:property>
+  <!-- Instantiate kopterworx mechanics "mechanics" -->
 	<xacro:include filename="$(find ardupilot_gazebo)/models/kopterworx/urdf/kopterworx_base.urdf.xacro" />
   <xacro:include filename="$(find rotors_description)/urdf/component_snippets.xacro" />
-  	<xacro:ardupilot
+	<!-- Ardupilot plugin -->
+  <xacro:ardupilot
 		imu_topic="/kopterworx/imu"
 		control_topic="/gazebo/command/motor_speed"
@@ -15,3 +20,40 @@
 		thrust_multiplier="600">
 	</xacro:ardupilot>
+	<xacro:if value="${enable_velodyne}">
+		<xacro:include filename="$(find velodyne_description)/urdf/VU-8.urdf.xacro"/>
+		<VU-8 parent="base_link" name="velodyne" topic="${namespace}/velodyne_points" hz="20" samples="440" gpu="false"
+						min_range="1" lasers="16">
+				<xacro:insert_block name="horizontal_velodyne_origin"/>
+		</VU-8>
+	</xacro:if>
+	<!-- Realistic odometry sensor with noise -->
+	<xacro:odometry_plugin_macro
+		namespace="${namespace}"
+		odometry_sensor_suffix=""
+		parent_link="base_link"
+		pose_topic="pose"
+		pose_with_covariance_topic="pose_with_covariance"
+		position_topic="position"
+		transform_topic="transform"
+		odometry_topic="odometry"
+		parent_frame_id="world"
+		child_frame_id="${namespace}/base_link"
+		mass_odometry_sensor="0.01"
+		measurement_divisor="20"
+		measurement_delay="0"
+		unknown_delay="0.0"
+		noise_normal_position="0.0 0.0 0.0"
+		noise_normal_quaternion="0.0 0.0 0.0"
+		noise_normal_linear_velocity="0.0 0.0 0.0"
+		noise_normal_angular_velocity="0.0 0.0 0.0"
+		noise_uniform_position="0.0 0.0 0.0"
+		noise_uniform_quaternion="0.0 0.0 0.0"
+		noise_uniform_linear_velocity="0.0 0.0 0.0"
+		noise_uniform_angular_velocity="0.0 0.0 0.0"
+		enable_odometry_map="false"
+		odometry_map=""
+		image_scale="">
+		<inertia ixx="0.00001" ixy="0.0" ixz="0.0" iyy="0.00001" iyz="0.0" izz="0.00001" /> <!-- [kg m^2] [kg m^2] [kg m^2] [kg m^2] [kg m^2] [kg m^2] -->
+		<origin xyz="0.0 0.0 0.0" rpy="0.0 0.0 0.0" />
+	</xacro:odometry_plugin_macro>
 </robot>

Commit message: [kopterworx.urdf.xacro] Add camera properties and macro.

File: models/kopterworx/urdf/kopterworx.urdf.xacro (robot description, xacro)
@@ -6,4 +6,19 @@
     <origin xyz="0.08 0. -0.1578" rpy="3.141592653589793 0.1323284641020683 0." />
 	</xacro:property>
+	<xacro:property name="front_facing_camera">
+		<origin xyz="0.2 0 0.05" rpy="0 0 0"/>
+	</xacro:property>
+	<xacro:property name="down_facing_camera">
+	  <origin xyz="0 0.2 -0.3" rpy="-1.570796 1.570796 0"/>
+	</xacro:property>
+  <xacro:property name="camera_mass" value="1e-5"/>
+	<xacro:property name="camera_size" value="0.05" />
+  <xacro:property name="camera_inertia">
+    <inertia
+    ixx="1e-12"
+    iyy="1e-12"
+    izz="1e-12"
+    ixy="0.0" ixz="0.0" iyz="0.0" />
+  </xacro:property>
   <!-- Instantiate kopterworx mechanics "mechanics" -->
 	<xacro:include filename="$(find ardupilot_gazebo)/models/kopterworx/urdf/kopterworx_base.urdf.xacro" />
@@ -57,3 +72,11 @@
 		<origin xyz="0.0 0.0 0.0" rpy="0.0 0.0 0.0" />
 	</xacro:odometry_plugin_macro>
+  <xacro:cam
+    namespace="$(arg namespace)"
+    camera_link="${camera_size}"
+    camera_mass="${camera_mass}"
+    parent="base_link">
+		<xacro:insert_block name="front_facing_camera"/>
+    <xacro:insert_block name="camera_inertia"/>
+  </xacro:cam>
 </robot>

Commit message: Add gimbal with RBGD camera on kopterworx

File: models/kopterworx/urdf/kopterworx.urdf.xacro (robot description, xacro)
@@ -76,4 +76,5 @@
 		<origin xyz="0.0 0.0 0.0" rpy="0.0 0.0 0.0" />
 	</xacro:odometry_plugin_macro>
+<!-- Choose one of the following (and comment out the other): fixed RGBD camera or gimbal with RGBD camera. -->
   <xacro:cam
     namespace="$(arg namespace)"
@@ -84,3 +85,6 @@
     <xacro:insert_block name="camera_inertia"/>
   </xacro:cam>
+<!--   <xacro:gimbal_macro parent="base_link">
+    <origin xyz="0.25 0 -0.1" rpy="0 0 0"/>
+  </xacro:gimbal_macro> -->
 </robot>

File: models/util/multirotor_base.urdf.xacro (robot description, xacro)
@@ -285,3 +285,173 @@
     </gazebo>
   </xacro:macro>
+  <!-- We add a <transmission> block for every joint that we wish to actuate. -->
+  <xacro:macro name="transmisija" params="trans_number joint_name">
+    <transmission name="transmission_${trans_number}">
+      <type>transmission_interface/SimpleTransmission</type>
+      <joint name="${joint_name}">
+        <hardwareInterface>hardware_interface/EffortJointInterface</hardwareInterface>
+      </joint>
+      <actuator name="motor_${trans_number}">
+        <hardwareInterface>hardware_interface/EffortActuatorInterface</hardwareInterface>
+        <mechanicalReduction>1</mechanicalReduction>
+      </actuator>
+    </transmission>
+  </xacro:macro>
+  <xacro:macro name="gimbal_macro" params="parent *origin">
+        <joint name="gimbal_position" type="fixed">
+            <xacro:insert_block name="origin"/>
+            <parent link="base_link"/>
+            <child link="gimbal_link_1"/>
+        </joint>
+        <gazebo reference="gimbal_position">
+            <preserveFixedJoint>true</preserveFixedJoint>
+        </gazebo>
+        <link name="gimbal_link_1">
+            <inertial>
+                <mass value="0.0001" />
+                <origin xyz="0 0 0" rpy="0 0 0" />
+                <inertia ixx="0.0001" ixy="0" ixz="0" iyy="0.0001" iyz="0" izz="0.0001" />
+            </inertial>
+<!--             <visual>
+                <geometry>
+                <box size="0.01 0.01 0.01" />
+                </geometry>
+            </visual> -->
+        </link>
+        <joint name="gimbal_yaw_joint" type="continuous">
+            <parent link="gimbal_link_1" />
+            <child link="gimbal_link_2" />
+            <axis xyz="0 0 1" />
+            <dynamics damping="0.0" friction="0.0" />
+        </joint>
+        <link name="gimbal_link_2">
+            <inertial>
+                <mass value="0.0001" />
+                <origin xyz="0 0 0" rpy="0 0 0" />
+                <inertia ixx="0.0001" ixy="0" ixz="0" iyy="0.0001" iyz="0" izz="0.0001" />
+            </inertial>
+            <visual>
+                <geometry>
+                <box size="0.01 0.01 0.01" />
+                </geometry>
+            </visual>
+        </link>
+        <joint name="gimbal_pitch_joint" type="continuous">
+            <parent link="gimbal_link_2" />
+            <child link="gimbal_link_3" />
+            <axis xyz="0 1 0" />
+            <dynamics damping="0.0" friction="0.0" />
+        </joint>
+        <link name="gimbal_link_3">
+            <inertial>
+                <mass value="0.0001" />
+                <origin xyz="0 0 0" rpy="0 0 0" />
+                <inertia ixx="0.0001" ixy="0" ixz="0" iyy="0.0001" iyz="0" izz="0.0001" />
+            </inertial>
+ <!--            <visual>
+                <geometry>
+                <box size="0.01 0.01 0.01" />
+                </geometry>
+            </visual> -->
+        </link>
+        <joint name="gimbal_roll_joint" type="continuous">
+            <parent link="gimbal_link_3" />
+            <child link="gimbal_link_4" />
+            <axis xyz="1 0 0" />
+            <dynamics damping="0.0" friction="0.0" />
+        </joint>
+        <link name="gimbal_link_4">
+            <inertial>
+                <mass value="0.0001" />
+                <origin xyz="0 0 0" rpy="0 0 ${-pi}" />
+                <inertia ixx="0.0001" ixy="0" ixz="0" iyy="0.0001" iyz="0" izz="0.0001" />
+            </inertial>
+<!--             <visual>
+                <geometry>
+                <box size="0.01 0.01 0.01" />
+                </geometry>
+            </visual> -->
+        </link>
+        <joint name="camera_gimbal_joint" type="continuous">
+            <parent link="gimbal_link_4" />
+            <child link="camera_link" />
+            <axis xyz="0 0 1" />
+            <dynamics damping="0.0" friction="0.0" />
+        </joint>
+        <link name="camera_link">
+        </link>
+        <joint name="camera_optical_joint" type="fixed">
+            <origin xyz="0 0 0" rpy="${-pi/2} 0.0 ${-pi/2}" />
+            <parent link="camera_link" />
+            <child link="camera_optical_frame"/>
+        </joint>
+        <gazebo reference="camera_optical_joint">
+            <preserveFixedJoint>true</preserveFixedJoint>
+        </gazebo>
+        <link name="camera_optical_frame">
+        </link>
+        <gazebo reference="gimbal_link_4">
+            <sensor type="depth" name="camera">
+              <update_rate>50.0</update_rate>
+              <camera name="head">
+                <horizontal_fov>1.5707963268</horizontal_fov>
+                <image>
+                  <width>1280</width>
+                  <height>720</height>
+                  <format>R8G8B8</format>
+                </image>
+                <clip>
+                  <near>0.02</near>
+                  <far>300</far>
+                </clip>
+                <noise>
+                  <type>gaussian</type>
+                  <mean>0.0</mean>
+                  <stddev>0.007</stddev>
+                </noise>
+              </camera>
+              <plugin name="camera_plugin" filename="libgazebo_ros_openni_kinect.so">
+                <baseline>0.2</baseline>
+                <alwaysOn>true</alwaysOn>
+                <!-- Keep this zero, update_rate in the parent <sensor> tag
+                  will control the frame rate. -->
+                <updateRate>0.0</updateRate>
+                <cameraName>${namespace}/camera_ir</cameraName>
+                <imageTopicName>/${namespace}/camera/color/image_raw</imageTopicName>
+                <cameraInfoTopicName>/${namespace}/camera/color/camera_info</cameraInfoTopicName>
+                <depthImageTopicName>/${namespace}/camera/depth/image_raw</depthImageTopicName>
+                <depthImageCameraInfoTopicName>/${namespace}/camera/depth/camera_info</depthImageCameraInfoTopicName>
+                <pointCloudTopicName>/${namespace}/camera/depth/points</pointCloudTopicName>
+                <frameName>camera_optical_frame</frameName>
+                <pointCloudCutoff>2.0</pointCloudCutoff>
+                <pointCloudCutoffMax>15.0</pointCloudCutoffMax>
+                <distortionK1>0</distortionK1>
+                <distortionK2>0</distortionK2>
+                <distortionK3>0</distortionK3>
+                <distortionT1>0</distortionT1>
+                <distortionT2>0</distortionT2>
+                <CxPrime>0</CxPrime>
+                <Cx>0</Cx>
+                <Cy>0</Cy>
+                <focalLength>0</focalLength>
+                <hackBaseline>0</hackBaseline>
+              </plugin>
+            </sensor>
+        </gazebo>
+        <gazebo>
+          <plugin name="gimbal_controller" filename="libGazeboGimbalPlugin.so"/>
+        </gazebo>
+        <xacro:transmisija
+          trans_number="g1"
+          joint_name="gimbal_roll_joint">
+        </xacro:transmisija>
+        <xacro:transmisija
+          trans_number="g2"
+          joint_name="gimbal_pitch_joint">
+        </xacro:transmisija>
+        <xacro:transmisija
+          trans_number="g3"
+          joint_name="gimbal_yaw_joint">
+        </xacro:transmisija>
+    </xacro:macro>
 </robot>

Commit message: Add Rotating Velodyne urdf

File: models/kopterworx/urdf/kopterworx.urdf.xacro (robot description, xacro)
@@ -3,8 +3,16 @@
   <xacro:property name="namespace" value="$(arg namespace)" />
   <xacro:property name="enable_velodyne" value="$(arg enable_velodyne)"/>
+	<xacro:property name="enable_rotating_velodyne" value="$(arg enable_rotating_velodyne)" />
 	<xacro:property name="fdm_port_in" value="$(arg fdm_port_in)"/>
 	<xacro:property name="fdm_port_out" value="$(arg fdm_port_out)"/>
+	<gazebo>
+    <plugin name="gazebo_ros_control" filename="libgazebo_ros_control.so">
+      <robotNamespace>/$(arg namespace)</robotNamespace>
+      <robotParam>/$(arg namespace)/robot_description </robotParam>
+      <robotSimType>gazebo_ros_control/DefaultRobotHWSim</robotSimType>
+    </plugin>
+  </gazebo>
 	<xacro:property name="horizontal_velodyne_origin">
-    <origin xyz="0.08 0. -0.1578" rpy="3.141592653589793 0.1323284641020683 0." />
+    <origin xyz="0.08 0. -0.1578" rpy="-3.141592653589793 0.1323284641020683 0." />
 	</xacro:property>
 	<xacro:property name="front_facing_camera">
@@ -40,9 +48,18 @@
 	</xacro:ardupilot>
 	<xacro:if value="${enable_velodyne}">
-		<xacro:include filename="$(find velodyne_description)/urdf/VU-8.urdf.xacro"/>
-		<VU-8 parent="base_link" name="velodyne" topic="${namespace}/velodyne_points" hz="10" samples="440" gpu="false"
-						min_range="1" lasers="16">
-				<xacro:insert_block name="horizontal_velodyne_origin"/>
-		</VU-8>
+		<xacro:if value="${enable_rotating_velodyne}">
+			<xacro:include filename="$(find velodyne_description)/urdf/VU-8.urdf-rotating.xacro"/>
+			<VU-8 parent="base_link_inertia" name="velodyne" topic="${namespace}/velodyne_points" hz="10" samples="440" gpu="false"
+							min_range="1" max_range="50" lasers="16">
+					<xacro:insert_block name="horizontal_velodyne_origin"/>
+			</VU-8>
+		</xacro:if>
+		<xacro:unless value="${enable_rotating_velodyne}">
+			<xacro:include filename="$(find velodyne_description)/urdf/VU-8.urdf.xacro"/>
+			<VU-8 parent="base_link_inertia" name="velodyne" topic="${namespace}/velodyne_points" hz="10" samples="440" gpu="false"
+							min_range="1" max_range="50" lasers="16">
+					<xacro:insert_block name="horizontal_velodyne_origin"/>
+			</VU-8>
+		</xacro:unless>
 	</xacro:if>
 	<!-- Realistic odometry sensor with noise -->

Commit message: [kopterworx] Add argument for max range

File: models/kopterworx/urdf/kopterworx.urdf.xacro (robot description, xacro)
@@ -6,4 +6,5 @@
 	<xacro:property name="fdm_port_in" value="$(arg fdm_port_in)"/>
 	<xacro:property name="fdm_port_out" value="$(arg fdm_port_out)"/>
+	<xacro:property name="max_range" value="$(arg max_range)"/>
 	<gazebo>
     <plugin name="gazebo_ros_control" filename="libgazebo_ros_control.so">
@@ -51,5 +52,5 @@
 			<xacro:include filename="$(find velodyne_description)/urdf/VU-8.urdf-rotating.xacro"/>
 			<VU-8 parent="base_link_inertia" name="velodyne" topic="${namespace}/velodyne_points" hz="10" samples="440" gpu="false"
-							min_range="1" max_range="50" lasers="16">
+							min_range="1" max_range="${max_range}" lasers="16">
 					<xacro:insert_block name="horizontal_velodyne_origin"/>
 			</VU-8>
@@ -58,5 +59,5 @@
 			<xacro:include filename="$(find velodyne_description)/urdf/VU-8.urdf.xacro"/>
 			<VU-8 parent="base_link_inertia" name="velodyne" topic="${namespace}/velodyne_points" hz="10" samples="440" gpu="false"
-							min_range="1" max_range="50" lasers="16">
+							min_range="1" max_range="${max_range}" lasers="16">
 					<xacro:insert_block name="horizontal_velodyne_origin"/>
 			</VU-8>

Commit message: Add prefix to base_link lmark1/uav_ros_simulation#8

File: models/kopterworx/urdf/kopterworx.urdf.xacro (robot description, xacro)
@@ -68,5 +68,5 @@
 		namespace="${namespace}"
 		odometry_sensor_suffix=""
-		parent_link="base_link"
+		parent_link="${namespace}/base_link"
 		pose_topic="pose"
 		pose_with_covariance_topic="pose_with_covariance"
@@ -99,5 +99,5 @@
     camera_link="${camera_size}"
     camera_mass="${camera_mass}"
-    parent="base_link">
+    parent="${namespace}/base_link">
 		<xacro:insert_block name="front_facing_camera"/>
     <xacro:insert_block name="camera_inertia"/>

File: models/kopterworx/urdf/kopterworx_base.urdf.xacro (robot description, xacro)
@@ -54,5 +54,5 @@
     motor_constant="${motor_constant}"
     moment_constant="${moment_constant}"
-    parent="base_link"
+    parent="$(arg namespace)/base_link"
     mass_rotor="${mass_rotor}"
     radius_rotor="${radius_rotor}"
@@ -74,5 +74,5 @@
     motor_constant="${motor_constant}"
     moment_constant="${moment_constant}"
-    parent="base_link"
+    parent="$(arg namespace)/base_link"
     mass_rotor="${mass_rotor}"
     radius_rotor="${radius_rotor}"
@@ -94,5 +94,5 @@
     motor_constant="${motor_constant}"
     moment_constant="${moment_constant}"
-    parent="base_link"
+    parent="$(arg namespace)/base_link"
     mass_rotor="${mass_rotor}"
     radius_rotor="${radius_rotor}"
@@ -114,5 +114,5 @@
     motor_constant="${motor_constant}"
     moment_constant="${moment_constant}"
-    parent="base_link"
+    parent="$(arg namespace)/base_link"
     mass_rotor="${mass_rotor}"
     radius_rotor="${radius_rotor}"
@@ -128,5 +128,5 @@
     <xacro:insert_block name="rotor_inertia" />
   </xacro:vertical_rotor>
-  <gazebo reference="base_link">
+  <gazebo reference="$(arg namespace)/base_link">
     <dampingFactor>0.001</dampingFactor>
   </gazebo>

File: models/util/multirotor_base.urdf.xacro (robot description, xacro)
@@ -18,8 +18,8 @@
   <xacro:macro name="multirotor_base_macro"
     params="robot_namespace mass body_width body_height mesh_file mesh_scale *origin *inertia">
-    <link name="base_link"></link>
+    <link name="${robot_namespace}/base_link"></link>
     <joint name="base_joint" type="fixed">
       <xacro:insert_block name="origin"/>
-      <parent link="base_link" />
+      <parent link="${robot_namespace}/base_link" />
       <child link="base_link_inertia" />
     </joint>
@@ -76,5 +76,5 @@
     <!-- IMU joint -->
     <joint name="imu_joint" type="revolute">
-      <parent link="base_link" />
+      <parent link="${robot_namespace}/base_link" />
       <child link="imu_link" />
       <limit upper="0" lower="0" effort="0" velocity="0" />
@@ -84,5 +84,5 @@
       <plugin filename="librotors_gazebo_multirotor_base_plugin.so" name="rosbag">
         <robotNamespace>${robot_namespace}</robotNamespace>
-        <linkName>base_link</linkName>
+        <linkName>${robot_namespace}/base_link</linkName>
         <rotorVelocitySlowdownSim>${rotor_velocity_slowdown_sim}</rotorVelocitySlowdownSim>
       </plugin>
