Commit message: Finish lmark1/uav_ros_simulation#8

File: models/kopterworx/urdf/kopterworx.urdf.xacro (robot description, xacro)
@@ -40,8 +40,8 @@
 		control_topic="/${namespace}/gazebo/command/motor_speed"
 		imu_sensor_name="${namespace}::imu_link::imu_sensor"
-		rotor_0_joint="${namespace}::rotor_0_joint"
-		rotor_1_joint="${namespace}::rotor_1_joint"
-		rotor_2_joint="${namespace}::rotor_2_joint"
-		rotor_3_joint="${namespace}::rotor_3_joint"
+		rotor_0_joint="${namespace}::${namespace}/rotor_0_joint"
+		rotor_1_joint="${namespace}::${namespace}/rotor_1_joint"
+		rotor_2_joint="${namespace}::${namespace}/rotor_2_joint"
+		rotor_3_joint="${namespace}::${namespace}/rotor_3_joint"
 		thrust_multiplier="600"
 		fdm_port_in="${fdm_port_in}"

File: models/util/multirotor_base.urdf.xacro (robot description, xacro)
@@ -22,7 +22,7 @@
       <xacro:insert_block name="origin"/>
       <parent link="${robot_namespace}/base_link" />
-      <child link="base_link_inertia" />
+      <child link="${robot_namespace}/base_link_inertia" />
     </joint>
-    <link name="base_link_inertia">
+    <link name="${robot_namespace}/base_link_inertia">
       <inertial>
         <mass value="${mass}" />  <!-- [kg] -->
@@ -92,5 +92,5 @@
   <xacro:macro name="vertical_rotor"
     params="robot_namespace suffix direction motor_constant moment_constant parent mass_rotor radius_rotor time_constant_up time_constant_down max_rot_velocity motor_number rotor_drag_coefficient rolling_moment_coefficient color prop_scale *origin *inertia">
-    <joint name="rotor_${motor_number}_joint" type="continuous">
+    <joint name="${robot_namespace}/rotor_${motor_number}_joint" type="continuous">
       <xacro:insert_block name="origin" />
       <axis xyz="0 0 1" />
@@ -98,10 +98,10 @@
       <!-- <limit effort="2000" velocity="${max_rot_velocity}" /> -->
       <parent link="${parent}" />
-      <child link="rotor_${motor_number}" />
+      <child link="${robot_namespace}/rotor_${motor_number}" />
     </joint>
     <!-- TODO(ff): not currently set because it's not yet supported -->
     <!-- <gazebo reference="rotor_${motor_number}_joint"> <axis> <xyz>0 0 1</xyz>
       <limit> <velocity> ${max_rot_velocity} </velocity> </limit> </axis> </gazebo> -->
-    <link name="rotor_${motor_number}">
+    <link name="${robot_namespace}/rotor_${motor_number}">
       <inertial>
         <mass value="${mass_rotor}" /> <!-- [kg] -->
@@ -124,6 +124,6 @@
     <gazebo>
       <plugin name="${suffix}_motor_model" filename="librotors_gazebo_motor_model.so">
-        <jointName>rotor_${motor_number}_joint</jointName>
-        <linkName>rotor_${motor_number}</linkName>
+        <jointName>${robot_namespace}/rotor_${motor_number}_joint</jointName>
+        <linkName>${robot_namespace}/rotor_${motor_number}</linkName>
         <turningDirection>${direction}</turningDirection>
         <timeConstantUp>${time_constant_up}</timeConstantUp>
@@ -140,5 +140,5 @@
       </plugin>
     </gazebo>
-    <gazebo reference="rotor_${motor_number}">
+    <gazebo reference="${robot_namespace}/rotor_${motor_number}">
       <material>Gazebo/${color}</material>
     </gazebo>
@@ -210,5 +210,5 @@
   <xacro:macro name="cam" params="namespace camera_link camera_mass parent *origin *inertia">
     <!-- Camera link -->
-    <link name="camera_box">
+    <link name="${namespace}/camera_box">
       <!--collision>
         <origin xyz="0 0 0" rpy="0 0 0"/>
@@ -233,14 +233,14 @@
       <xacro:insert_block name="origin"/>
       <parent link="${parent}"/>
-      <child link="camera_box"/>
+      <child link="${namespace}/camera_box"/>
     </joint>
-    <link name="camera"/>
+    <link name="${namespace}/camera"/>
     <joint name="camera_help" type="fixed">
-      <parent link="camera_box"/>
-      <child link="camera"/>
+      <parent link="${namespace}/camera_box"/>
+      <child link="${namespace}/camera"/>
       <origin rpy="-1.57 0 -1.57"/>
     </joint>
     <!-- camera -->
-    <gazebo reference="camera_box">
+    <gazebo reference="${namespace}/camera_box">
       <sensor type="depth" name="camera">
         <update_rate>30.0</update_rate>
@@ -274,5 +274,5 @@
           <depthImageCameraInfoTopicName>/${namespace}/camera/depth/camera_info</depthImageCameraInfoTopicName>
           <pointCloudTopicName>/${namespace}/camera/depth_registered/points</pointCloudTopicName>
-          <frameName>camera</frameName>
+          <frameName>${namespace}/camera</frameName>
           <pointCloudCutoff>0.3</pointCloudCutoff>
           <pointCloudCutoffMax>10.0</pointCloudCutoffMax>

Commit message: [kopterworx] Add remap_gazebo_tf and laser_count parameters

File: models/kopterworx/urdf/kopterworx.urdf.xacro (robot description, xacro)
@@ -7,4 +7,5 @@
 	<xacro:property name="fdm_port_out" value="$(arg fdm_port_out)"/>
 	<xacro:property name="max_range" value="$(arg max_range)"/>
+	<xacro:property name="laser_count" value="$(arg laser_count)"/>
 	<gazebo>
     <plugin name="gazebo_ros_control" filename="libgazebo_ros_control.so">
@@ -35,5 +36,8 @@
 	<xacro:include filename="$(find ardupilot_gazebo)/models/kopterworx/urdf/kopterworx_base.urdf.xacro" />
   <xacro:include filename="$(find rotors_description)/urdf/component_snippets.xacro" />
-	<!-- Ardupilot plugin -->
+  <!-- Ardupilot plugin
+    NOTE: thrust_multiplier
+      Value is tuned in order for mavros/setpoint_raw/attitude/thrust to reflect real-world behavior.
+  -->
   <xacro:ardupilot
 		imu_topic="/${namespace}/imu"
@@ -60,5 +64,5 @@
 				min_range="1"
 				max_range="${max_range}"
-				lasers="16">
+				lasers="32">
 				<xacro:insert_block name="horizontal_velodyne_origin"/>
 			</xacro:lidar-x>
@@ -75,5 +79,5 @@
 				min_range="1"
 				max_range="${max_range}"
-				lasers="16">
+				lasers="32">
 				<xacro:insert_block name="horizontal_velodyne_origin"/>
 			</xacro:lidar-x>

Commit message: Add magnet plugin

File: models/kopterworx/urdf/kopterworx.urdf.xacro (robot description, xacro)
@@ -3,4 +3,5 @@
   <xacro:property name="namespace" value="$(arg namespace)" />
   <xacro:property name="enable_velodyne" value="$(arg enable_velodyne)"/>
+  <xacro:property name="enable_magnet" value="$(arg enable_magnet)"/>
 	<xacro:property name="enable_rotating_velodyne" value="$(arg enable_rotating_velodyne)" />
 	<xacro:property name="fdm_port_in" value="$(arg fdm_port_in)"/>
@@ -52,4 +53,15 @@
 		fdm_port_out="${fdm_port_out}">
 	</xacro:ardupilot>
+  <xacro:if value="${enable_magnet}">
+    <xacro:magnet_plugin
+      parent="${namespace}/base_link_inertia"
+      namespace="${namespace}"
+      name="uav_magnet"
+      moment_x="0"
+      moment_y="0"
+      moment_z="50"
+      length="0.25">
+    </xacro:magnet_plugin>
+  </xacro:if>
 	<xacro:if value="${enable_velodyne}">
 		<xacro:if value="${enable_rotating_velodyne}">

File: models/util/multirotor_base.urdf.xacro (robot description, xacro)
@@ -461,3 +461,60 @@
         </xacro:transmisija>
     </xacro:macro>
+    <xacro:macro name="magnet_plugin" params="parent namespace name moment_x moment_y moment_z length">
+      <joint name="${namespace}/electromagnet_joint" type="fixed">
+        <axis xyz="0 1 0" />
+        <origin xyz="0 0 ${-length}" rpy="0 0 0" />
+        <parent link="${parent}"/>
+        <child link="${namespace}/electromagnet_actuator"/>
+      </joint>
+      <joint name="${namespace}/electromagnet_joint_bar" type="fixed">
+        <axis xyz="0 1 0" />
+        <origin xyz="0 0 ${length/2}" rpy="0 0 0"/>
+        <parent link="${namespace}/electromagnet_actuator"/>
+        <child link="${namespace}/electromagnet_bar"/>
+      </joint>
+      <link name="${namespace}/electromagnet_bar">
+        <inertial>
+          <origin xyz="0 0 0" rpy="0 0 0" />
+          <mass value="0.00025"/>
+          <inertia ixx="0.000001" ixy="0" ixz="0" iyy="0.000001" iyz="0" izz="0.000001" />
+        </inertial>
+        <visual>
+          <geometry>
+            <cylinder radius="0.01" length="${length}"/>
+          </geometry>
+        </visual>
+      </link>
+      <link name="${namespace}/electromagnet_actuator">
+        <inertial>
+          <origin xyz="0 0 0" rpy="0 0 0" />
+          <mass value="0.025"/>
+          <inertia ixx="0.0001" ixy="0" ixz="0" iyy ="0.0001" iyz = "0" izz = "0.0001" />
+        </inertial>
+        <collision name="collision">
+          <geometry>
+            <cylinder radius="0.04" length="0.035"/>
+          </geometry>
+        </collision>
+        <visual>
+          <geometry>
+            <cylinder radius="0.08" length="0.035"/>
+          </geometry>
+        </visual>
+      </link>
+       <gazebo reference="${namespace}/electromagnet_actuator">
+        <material>Gazebo/Green</material>
+      </gazebo>
+      <gazebo>
+        <plugin name="dipole_magnet" filename="libstorm_gazebo_dipole_magnet.so">
+          <bodyName>${namespace}/electromagnet_actuator</bodyName>
+          <dipole_moment>${moment_x} ${moment_y} ${moment_z}</dipole_moment>
+          <!-- Set to false if not using ROS -->
+          <shouldPublish>true</shouldPublish>
+          <topicNs>${name}</topicNs>
+          <updateRate>100</updateRate>
+          <gain>1.0</gain>
+        </plugin>
+      </gazebo>
+    </xacro:macro>
 </robot>

Commit message: Update Magnet macro

File: models/kopterworx/urdf/kopterworx.urdf.xacro (robot description, xacro)
@@ -61,5 +61,6 @@
       moment_y="0"
       moment_z="50"
-      length="0.25">
+      length="0.25"
+      offset="0.07">
     </xacro:magnet_plugin>
   </xacro:if>

File: models/util/multirotor_base.urdf.xacro (robot description, xacro)
@@ -461,5 +461,5 @@
         </xacro:transmisija>
     </xacro:macro>
-    <xacro:macro name="magnet_plugin" params="parent namespace name moment_x moment_y moment_z length">
+    <xacro:macro name="magnet_plugin" params="parent namespace name moment_x moment_y moment_z length offset">
       <joint name="${namespace}/electromagnet_joint" type="fixed">
         <axis xyz="0 1 0" />
@@ -482,5 +482,5 @@
         <visual>
           <geometry>
-            <cylinder radius="0.01" length="${length}"/>
+            <cylinder radius="0.01" length="${length + offset}"/>
           </geometry>
         </visual>
@@ -494,5 +494,5 @@
         <collision name="collision">
           <geometry>
-            <cylinder radius="0.04" length="0.035"/>
+            <cylinder radius="0.08" length="0.035"/>
           </geometry>
         </collision>
@@ -501,4 +501,5 @@
             <cylinder radius="0.08" length="0.035"/>
           </geometry>
+          <origin xyz="0 0 ${-offset/2}" rpy="0 0 0" />
         </visual>
       </link>
@@ -512,5 +513,5 @@
           <!-- Set to false if not using ROS -->
           <shouldPublish>true</shouldPublish>
-          <topicNs>${name}</topicNs>
+          <topicNs>${namespace}/${name}</topicNs>
           <updateRate>100</updateRate>
           <gain>1.0</gain>

Commit message: Add prefix to base_link for gimbal

File: models/kopterworx/urdf/kopterworx.urdf.xacro (robot description, xacro)
@@ -136,6 +136,8 @@
     <xacro:insert_block name="camera_inertia"/>
   </xacro:cam>
-<!--   <xacro:gimbal_macro parent="base_link">
-    <origin xyz="0.25 0 -0.1" rpy="0 0 0"/>
-  </xacro:gimbal_macro> -->
+	<!-- <xacro:gimbal_macro
+		namespace="$(arg namespace)"
+		parent="${namespace}/base_link">
+	<origin xyz="0.25 0 -0.1" rpy="0 0 0"/>
+	</xacro:gimbal_macro> -->
 </robot>

File: models/util/multirotor_base.urdf.xacro (robot description, xacro)
@@ -304,8 +304,8 @@
     </transmission>
   </xacro:macro>
-  <xacro:macro name="gimbal_macro" params="parent *origin">
+  <xacro:macro name="gimbal_macro" params="namespace parent *origin">
         <joint name="gimbal_position" type="fixed">
             <xacro:insert_block name="origin"/>
-            <parent link="base_link"/>
+            <parent link="${namespace}/base_link"/>
             <child link="gimbal_link_1"/>
         </joint>

Commit message: [Launch,Models] Add collision bitmask argument option.

File: models/kopterworx/urdf/kopterworx.urdf.xacro (robot description, xacro)
@@ -9,4 +9,7 @@
 	<xacro:property name="max_range" value="$(arg max_range)"/>
 	<xacro:property name="laser_count" value="$(arg laser_count)"/>
+	<!-- Collision bitmask - By default collides with everything -->
+	<xacro:arg name="collision_bitmask" default="-1" />
+	<xacro:property name="collision_bitmask" value="$(arg collision_bitmask)" />
 	<gazebo>
     <plugin name="gazebo_ros_control" filename="libgazebo_ros_control.so">

File: models/kopterworx/urdf/kopterworx_base.urdf.xacro (robot description, xacro)
@@ -26,4 +26,7 @@
   <xacro:property name="rotor_drag_coefficient" value="8.06428e-05" />
   <xacro:property name="rolling_moment_coefficient" value="0.000001" />
+  <!-- Collision bitmask - By default collides with everything -->
+  <xacro:arg name="collision_bitmask" default="-1" />
+  <xacro:property name="collision_bitmask" value="$(arg collision_bitmask)" />
   <!-- Property Blocks -->
   <xacro:property name="body_inertia">
@@ -130,4 +133,11 @@
   <gazebo reference="$(arg namespace)/base_link">
     <dampingFactor>0.001</dampingFactor>
+    <collision>
+      <surface>
+        <contact>
+          <collide_bitmask>${collision_bitmask}</collide_bitmask>
+        </contact>
+      </surface>
+    </collision>
   </gazebo>
 </robot>

File: models/util/multirotor_base.urdf.xacro (robot description, xacro)
@@ -18,4 +18,13 @@
   <xacro:macro name="multirotor_base_macro"
     params="robot_namespace mass body_width body_height mesh_file mesh_scale *origin *inertia">
+    <gazebo reference="${robot_namespace}/base_link">
+      <collision>
+        <surface>
+          <contact>
+            <collide_bitmask>${collision_bitmask}</collide_bitmask>
+          </contact>
+        </surface>
+      </collision>
+    </gazebo>
     <link name="${robot_namespace}/base_link"></link>
     <joint name="base_joint" type="fixed">
@@ -24,4 +33,13 @@
       <child link="${robot_namespace}/base_link_inertia" />
     </joint>
+    <gazebo reference="${robot_namespace}/base_link_inertia">
+      <collision>
+        <surface>
+          <contact>
+            <collide_bitmask>${collision_bitmask}</collide_bitmask>
+          </contact>
+        </surface>
+      </collision>
+    </gazebo>
     <link name="${robot_namespace}/base_link_inertia">
       <inertial>
@@ -55,4 +73,11 @@
     </link>
     <gazebo reference="imu_link">
+      <collision>
+        <surface>
+          <contact>
+            <collide_bitmask>${collision_bitmask}</collide_bitmask>
+          </contact>
+        </surface>
+      </collision>
       <sensor name="imu_sensor" type="imu">
         <always_on>true</always_on>
@@ -103,4 +128,13 @@
     <!-- <gazebo reference="rotor_${motor_number}_joint"> <axis> <xyz>0 0 1</xyz>
       <limit> <velocity> ${max_rot_velocity} </velocity> </limit> </axis> </gazebo> -->
+    <gazebo reference="${robot_namespace}/rotor_${motor_number}">
+      <collision>
+        <surface>
+          <contact>
+            <collide_bitmask>${collision_bitmask}</collide_bitmask>
+          </contact>
+        </surface>
+      </collision>
+    </gazebo>
     <link name="${robot_namespace}/rotor_${motor_number}">
       <inertial>
@@ -210,4 +244,13 @@
   <xacro:macro name="cam" params="namespace camera_link camera_mass parent *origin *inertia">
     <!-- Camera link -->
+    <gazebo reference="${namespace}/camera_box">
+      <collision>
+        <surface>
+          <contact>
+            <collide_bitmask>${collision_bitmask}</collide_bitmask>
+          </contact>
+        </surface>
+      </collision>
+    </gazebo>
     <link name="${namespace}/camera_box">
       <!--collision>
@@ -235,4 +278,13 @@
       <child link="${namespace}/camera_box"/>
     </joint>
+    <gazebo reference="${namespace}/camera">
+      <collision>
+        <surface>
+          <contact>
+            <collide_bitmask>${collision_bitmask}</collide_bitmask>
+          </contact>
+        </surface>
+      </collision>
+    </gazebo>
     <link name="${namespace}/camera"/>
     <joint name="camera_help" type="fixed">
@@ -313,4 +365,13 @@
             <preserveFixedJoint>true</preserveFixedJoint>
         </gazebo>
+        <gazebo reference="gimbal_link_1">
+          <collision>
+            <surface>
+              <contact>
+                <collide_bitmask>${collision_bitmask}</collide_bitmask>
+              </contact>
+            </surface>
+          </collision>
+        </gazebo>
         <link name="gimbal_link_1">
             <inertial>
@@ -331,4 +392,13 @@
             <dynamics damping="0.0" friction="0.0" />
         </joint>
+        <gazebo reference="gimbal_link_2">
+          <collision>
+            <surface>
+              <contact>
+                <collide_bitmask>${collision_bitmask}</collide_bitmask>
+              </contact>
+            </surface>
+          </collision>
+        </gazebo>
         <link name="gimbal_link_2">
             <inertial>
@@ -349,4 +419,13 @@
             <dynamics damping="0.0" friction="0.0" />
         </joint>
+        <gazebo reference="gimbal_link_3">
+          <collision>
+            <surface>
+              <contact>
+                <collide_bitmask>${collision_bitmask}</collide_bitmask>
+              </contact>
+            </surface>
+          </collision>
+        </gazebo>
         <link name="gimbal_link_3">
             <inertial>
@@ -367,4 +446,13 @@
             <dynamics damping="0.0" friction="0.0" />
         </joint>
+        <gazebo reference="gimbal_link_4">
+          <collision>
+            <surface>
+              <contact>
+                <collide_bitmask>${collision_bitmask}</collide_bitmask>
+              </contact>
+            </surface>
+          </collision>
+        </gazebo>
         <link name="gimbal_link_4">
             <inertial>
@@ -392,4 +480,13 @@
             <dynamics damping="0.0" friction="0.0" />
         </joint>
+        <gazebo reference="camera_link">
+          <collision>
+            <surface>
+              <contact>
+                <collide_bitmask>${collision_bitmask}</collide_bitmask>
+              </contact>
+            </surface>
+          </collision>
+        </gazebo>
         <link name="camera_link">
         </link>
@@ -401,4 +498,13 @@
         <gazebo reference="camera_optical_joint">
             <preserveFixedJoint>true</preserveFixedJoint>
+        </gazebo>
+        <gazebo reference="camera_optical_frame">
+          <collision>
+            <surface>
+              <contact>
+                <collide_bitmask>${collision_bitmask}</collide_bitmask>
+              </contact>
+            </surface>
+          </collision>
         </gazebo>
         <link name="camera_optical_frame">
@@ -481,4 +587,13 @@
         <child link="${namespace}/electromagnet_bar"/>
       </joint>
+      <gazebo reference="${namespace}/electromagnet_bar">
+        <collision>
+          <surface>
+            <contact>
+              <collide_bitmask>${collision_bitmask}</collide_bitmask>
+            </contact>
+          </surface>
+        </collision>
+      </gazebo>
       <link name="${namespace}/electromagnet_bar">
         <inertial>
@@ -493,4 +608,13 @@
         </visual>
       </link>
+      <gazebo reference="${namespace}/electromagnet_actuator">
+        <collision>
+          <surface>
+            <contact>
+              <collide_bitmask>${collision_bitmask}</collide_bitmask>
+            </contact>
+          </surface>
+        </collision>
+      </gazebo>
       <link name="${namespace}/electromagnet_actuator">
         <inertial>
