Commit message: Add controllable gimbal

File: models/kopterworx/urdf/kopterworx.urdf.xacro (robot description, xacro)
@@ -4,13 +4,14 @@
   <xacro:property name="enable_velodyne" value="$(arg enable_velodyne)"/>
   <xacro:property name="enable_magnet" value="$(arg enable_magnet)"/>
-	<xacro:property name="enable_rotating_velodyne" value="$(arg enable_rotating_velodyne)" />
-	<xacro:property name="fdm_port_in" value="$(arg fdm_port_in)"/>
-	<xacro:property name="fdm_port_out" value="$(arg fdm_port_out)"/>
-	<xacro:property name="max_range" value="$(arg max_range)"/>
-	<xacro:property name="laser_count" value="$(arg laser_count)"/>
-	<!-- Collision bitmask - By default collides with everything -->
-	<xacro:arg name="collision_bitmask" default="-1" />
-	<xacro:property name="collision_bitmask" value="$(arg collision_bitmask)" />
-	<gazebo>
+  <xacro:property name="enable_gimbal" value="$(arg enable_gimbal)"/>
+  <xacro:property name="enable_rotating_velodyne" value="$(arg enable_rotating_velodyne)" />
+  <xacro:property name="fdm_port_in" value="$(arg fdm_port_in)"/>
+  <xacro:property name="fdm_port_out" value="$(arg fdm_port_out)"/>
+  <xacro:property name="max_range" value="$(arg max_range)"/>
+  <xacro:property name="laser_count" value="$(arg laser_count)"/>
+  <!-- Collision bitmask - By default collides with everything -->
+  <xacro:arg name="collision_bitmask" default="-1" />
+  <xacro:property name="collision_bitmask" value="$(arg collision_bitmask)" />
+  <gazebo>
     <plugin name="gazebo_ros_control" filename="libgazebo_ros_control.so">
       <robotNamespace>/$(arg namespace)</robotNamespace>
@@ -19,15 +20,15 @@
     </plugin>
   </gazebo>
-	<xacro:property name="horizontal_velodyne_origin">
+  <xacro:property name="horizontal_velodyne_origin">
     <origin xyz="0.08 0. -0.1578" rpy="-3.141592653589793 0.1323284641020683 0." />
-	</xacro:property>
-	<xacro:property name="front_facing_camera">
-		<origin xyz="0.2 0 0.05" rpy="0 0 0"/>
-	</xacro:property>
-	<xacro:property name="down_facing_camera">
-	  <origin xyz="0 0.2 -0.3" rpy="-1.570796 1.570796 0"/>
-	</xacro:property>
+  </xacro:property>
+  <xacro:property name="front_facing_camera">
+    <origin xyz="0.2 0 0.05" rpy="0 0 0"/>
+  </xacro:property>
+  <xacro:property name="down_facing_camera">
+    <origin xyz="0 0.2 -0.3" rpy="-1.570796 1.570796 0"/>
+  </xacro:property>
   <xacro:property name="camera_mass" value="1e-5"/>
-	<xacro:property name="camera_size" value="0.05" />
+  <xacro:property name="camera_size" value="0.05" />
   <xacro:property name="camera_inertia">
     <inertia
@@ -38,5 +39,5 @@
   </xacro:property>
   <!-- Instantiate kopterworx mechanics "mechanics" -->
-	<xacro:include filename="$(find ardupilot_gazebo)/models/kopterworx/urdf/kopterworx_base.urdf.xacro" />
+  <xacro:include filename="$(find ardupilot_gazebo)/models/kopterworx/urdf/kopterworx_base.urdf.xacro" />
   <xacro:include filename="$(find rotors_description)/urdf/component_snippets.xacro" />
   <!-- Ardupilot plugin
@@ -45,15 +46,15 @@
   -->
   <xacro:ardupilot
-		imu_topic="/${namespace}/imu"
-		control_topic="/${namespace}/gazebo/command/motor_speed"
-		imu_sensor_name="${namespace}::imu_link::imu_sensor"
-		rotor_0_joint="${namespace}::${namespace}/rotor_0_joint"
-		rotor_1_joint="${namespace}::${namespace}/rotor_1_joint"
-		rotor_2_joint="${namespace}::${namespace}/rotor_2_joint"
-		rotor_3_joint="${namespace}::${namespace}/rotor_3_joint"
-		thrust_multiplier="600"
-		fdm_port_in="${fdm_port_in}"
-		fdm_port_out="${fdm_port_out}">
-	</xacro:ardupilot>
+    imu_topic="/${namespace}/imu"
+    control_topic="/${namespace}/gazebo/command/motor_speed"
+    imu_sensor_name="${namespace}::imu_link::imu_sensor"
+    rotor_0_joint="${namespace}::${namespace}/rotor_0_joint"
+    rotor_1_joint="${namespace}::${namespace}/rotor_1_joint"
+    rotor_2_joint="${namespace}::${namespace}/rotor_2_joint"
+    rotor_3_joint="${namespace}::${namespace}/rotor_3_joint"
+    thrust_multiplier="600"
+    fdm_port_in="${fdm_port_in}"
+    fdm_port_out="${fdm_port_out}">
+  </xacro:ardupilot>
   <xacro:if value="${enable_magnet}">
     <xacro:magnet_plugin
@@ -68,79 +69,83 @@
     </xacro:magnet_plugin>
   </xacro:if>
-	<xacro:if value="${enable_velodyne}">
-		<xacro:if value="${enable_rotating_velodyne}">
-			<xacro:include filename="$(find velodyne_description)/urdf/LiDAR-X-rotating.urdf.xacro"/>
-			<xacro:lidar-x
-				parent="${namespace}/base_link_inertia"
-				name="velodyne"
-				topic="${namespace}/velodyne_points"
-				hz="10"
-				samples="440"
-				gpu="false"
-				min_range="1"
-				max_range="${max_range}"
-				lasers="32">
-				<xacro:insert_block name="horizontal_velodyne_origin"/>
-			</xacro:lidar-x>
-		</xacro:if>
-		<xacro:unless value="${enable_rotating_velodyne}">
-			<xacro:include filename="$(find velodyne_description)/urdf/LiDAR-X.urdf.xacro"/>
-			<xacro:lidar-x
-				parent="${namespace}/base_link_inertia"
-				name="velodyne"
-				topic="${namespace}/velodyne_points"
-				hz="10"
-				samples="440"
-				gpu="false"
-				min_range="1"
-				max_range="${max_range}"
-				lasers="32">
-				<xacro:insert_block name="horizontal_velodyne_origin"/>
-			</xacro:lidar-x>
-		</xacro:unless>
-	</xacro:if>
-	<!-- Realistic odometry sensor with noise -->
-	<xacro:odometry_plugin_macro
-		namespace="${namespace}"
-		odometry_sensor_suffix=""
-		parent_link="${namespace}/base_link"
-		pose_topic="pose"
-		pose_with_covariance_topic="pose_with_covariance"
-		position_topic="position"
-		transform_topic="transform"
-		odometry_topic="odometry"
-		parent_frame_id="world"
-		child_frame_id="${namespace}/base_link"
-		mass_odometry_sensor="0.01"
-		measurement_divisor="20"
-		measurement_delay="0"
-		unknown_delay="0.0"
-		noise_normal_position="0.0 0.0 0.0"
-		noise_normal_quaternion="0.0 0.0 0.0"
-		noise_normal_linear_velocity="0.0 0.0 0.0"
-		noise_normal_angular_velocity="0.0 0.0 0.0"
-		noise_uniform_position="0.0 0.0 0.0"
-		noise_uniform_quaternion="0.0 0.0 0.0"
-		noise_uniform_linear_velocity="0.0 0.0 0.0"
-		noise_uniform_angular_velocity="0.0 0.0 0.0"
-		enable_odometry_map="false"
-		odometry_map=""
-		image_scale="">
-		<inertia ixx="0.00001" ixy="0.0" ixz="0.0" iyy="0.00001" iyz="0.0" izz="0.00001" /> <!-- [kg m^2] [kg m^2] [kg m^2] [kg m^2] [kg m^2] [kg m^2] -->
-		<origin xyz="0.0 0.0 0.0" rpy="0.0 0.0 0.0" />
-	</xacro:odometry_plugin_macro>
-<!-- Choose one of the following (and comment out the other): fixed RGBD camera or gimbal with RGBD camera. -->
-  <xacro:cam
-    namespace="$(arg namespace)"
-    camera_link="${camera_size}"
-    camera_mass="${camera_mass}"
-    parent="${namespace}/base_link">
-		<xacro:insert_block name="front_facing_camera"/>
-    <xacro:insert_block name="camera_inertia"/>
-  </xacro:cam>
-	<!-- <xacro:gimbal_macro
-		namespace="$(arg namespace)"
-		parent="${namespace}/base_link">
-	<origin xyz="0.25 0 -0.1" rpy="0 0 0"/>
-	</xacro:gimbal_macro> -->
+  <xacro:if value="${enable_velodyne}">
+    <xacro:if value="${enable_rotating_velodyne}">
+      <xacro:include filename="$(find velodyne_description)/urdf/LiDAR-X-rotating.urdf.xacro"/>
+      <xacro:lidar-x
+        parent="${namespace}/base_link_inertia"
+        name="velodyne"
+        topic="${namespace}/velodyne_points"
+        hz="10"
+        samples="440"
+        gpu="false"
+        min_range="1"
+        max_range="${max_range}"
+        lasers="32">
+        <xacro:insert_block name="horizontal_velodyne_origin"/>
+      </xacro:lidar-x>
+    </xacro:if>
+    <xacro:unless value="${enable_rotating_velodyne}">
+      <xacro:include filename="$(find velodyne_description)/urdf/LiDAR-X.urdf.xacro"/>
+      <xacro:lidar-x
+        parent="${namespace}/base_link_inertia"
+        name="velodyne"
+        topic="${namespace}/velodyne_points"
+        hz="10"
+        samples="440"
+        gpu="false"
+        min_range="1"
+        max_range="${max_range}"
+        lasers="32">
+        <xacro:insert_block name="horizontal_velodyne_origin"/>
+      </xacro:lidar-x>
+    </xacro:unless>
+  </xacro:if>
+  <!-- Realistic odometry sensor with noise -->
+  <xacro:odometry_plugin_macro
+    namespace="${namespace}"
+    odometry_sensor_suffix=""
+    parent_link="${namespace}/base_link"
+    pose_topic="pose"
+    pose_with_covariance_topic="pose_with_covariance"
+    position_topic="position"
+    transform_topic="transform"
+    odometry_topic="odometry"
+    parent_frame_id="world"
+    child_frame_id="${namespace}/base_link"
+    mass_odometry_sensor="0.01"
+    measurement_divisor="20"
+    measurement_delay="0"
+    unknown_delay="0.0"
+    noise_normal_position="0.0 0.0 0.0"
+    noise_normal_quaternion="0.0 0.0 0.0"
+    noise_normal_linear_velocity="0.0 0.0 0.0"
+    noise_normal_angular_velocity="0.0 0.0 0.0"
+    noise_uniform_position="0.0 0.0 0.0"
+    noise_uniform_quaternion="0.0 0.0 0.0"
+    noise_uniform_linear_velocity="0.0 0.0 0.0"
+    noise_uniform_angular_velocity="0.0 0.0 0.0"
+    enable_odometry_map="false"
+    odometry_map=""
+    image_scale="">
+    <inertia ixx="0.00001" ixy="0.0" ixz="0.0" iyy="0.00001" iyz="0.0" izz="0.00001" /> <!-- [kg m^2] [kg m^2] [kg m^2] [kg m^2] [kg m^2] [kg m^2] -->
+    <origin xyz="0.0 0.0 0.0" rpy="0.0 0.0 0.0" />
+  </xacro:odometry_plugin_macro>
+  <!-- Choose one of the following (and comment out the other): fixed RGBD camera or gimbal with RGBD camera. -->
+  <xacro:unless value="${enable_gimbal}">
+    <xacro:cam
+      namespace="$(arg namespace)"
+      camera_link="${camera_size}"
+      camera_mass="${camera_mass}"
+      parent="${namespace}/base_link">
+      <xacro:insert_block name="front_facing_camera"/>
+      <xacro:insert_block name="camera_inertia"/>
+    </xacro:cam>
+  </xacro:unless>
+  <xacro:if value="${enable_gimbal}">
+    <xacro:gimbal_macro
+      namespace="$(arg namespace)"
+      parent="${namespace}/base_link">
+      <xacro:insert_block name="front_facing_camera"/>
+    </xacro:gimbal_macro>
+  </xacro:if>
 </robot>

File: models/util/multirotor_base.urdf.xacro (robot description, xacro)
@@ -357,13 +357,13 @@
   </xacro:macro>
   <xacro:macro name="gimbal_macro" params="namespace parent *origin">
-        <joint name="gimbal_position" type="fixed">
+        <joint name="${namespace}/gimbal_position" type="fixed">
             <xacro:insert_block name="origin"/>
-            <parent link="${namespace}/base_link"/>
-            <child link="gimbal_link_1"/>
+            <parent link="${parent}"/>
+            <child link="${namespace}/gimbal_link_1"/>
         </joint>
-        <gazebo reference="gimbal_position">
+        <gazebo reference="${namespace}/gimbal_position">
             <preserveFixedJoint>true</preserveFixedJoint>
         </gazebo>
-        <gazebo reference="gimbal_link_1">
+        <gazebo reference="${namespace}/gimbal_link_1">
           <collision>
             <surface>
@@ -374,5 +374,6 @@
           </collision>
         </gazebo>
-        <link name="gimbal_link_1">
+        <!-- yawing link -->
+        <link name="${namespace}/gimbal_link_1">
             <inertial>
                 <mass value="0.0001" />
@@ -380,17 +381,12 @@
                 <inertia ixx="0.0001" ixy="0" ixz="0" iyy="0.0001" iyz="0" izz="0.0001" />
             </inertial>
-<!--             <visual>
-                <geometry>
-                <box size="0.01 0.01 0.01" />
-                </geometry>
-            </visual> -->
         </link>
-        <joint name="gimbal_yaw_joint" type="continuous">
-            <parent link="gimbal_link_1" />
-            <child link="gimbal_link_2" />
+        <joint name="${namespace}/gimbal_yaw_joint" type="continuous">
+            <parent link="${namespace}/gimbal_link_1" />
+            <child link="${namespace}/gimbal_link_2" />
             <axis xyz="0 0 1" />
             <dynamics damping="0.0" friction="0.0" />
         </joint>
-        <gazebo reference="gimbal_link_2">
+        <gazebo reference="${namespace}/gimbal_link_2">
           <collision>
             <surface>
@@ -401,5 +397,5 @@
           </collision>
         </gazebo>
-        <link name="gimbal_link_2">
+        <link name="${namespace}/gimbal_link_2">
             <inertial>
                 <mass value="0.0001" />
@@ -407,17 +403,12 @@
                 <inertia ixx="0.0001" ixy="0" ixz="0" iyy="0.0001" iyz="0" izz="0.0001" />
             </inertial>
-            <visual>
-                <geometry>
-                <box size="0.01 0.01 0.01" />
-                </geometry>
-            </visual>
         </link>
-        <joint name="gimbal_pitch_joint" type="continuous">
-            <parent link="gimbal_link_2" />
-            <child link="gimbal_link_3" />
+        <joint name="${namespace}/gimbal_pitch_joint" type="continuous">
+            <parent link="${namespace}/gimbal_link_2" />
+            <child link="${namespace}/gimbal_link_3" />
             <axis xyz="0 1 0" />
             <dynamics damping="0.0" friction="0.0" />
         </joint>
-        <gazebo reference="gimbal_link_3">
+        <gazebo reference="${namespace}/gimbal_link_3">
           <collision>
             <surface>
@@ -428,5 +419,5 @@
           </collision>
         </gazebo>
-        <link name="gimbal_link_3">
+        <link name="${namespace}/gimbal_link_3">
             <inertial>
                 <mass value="0.0001" />
@@ -440,11 +431,11 @@
             </visual> -->
         </link>
-        <joint name="gimbal_roll_joint" type="continuous">
-            <parent link="gimbal_link_3" />
-            <child link="gimbal_link_4" />
+        <joint name="${namespace}/gimbal_roll_joint" type="continuous">
+            <parent link="${namespace}/gimbal_link_3" />
+            <child link="${namespace}/gimbal_link_4" />
             <axis xyz="1 0 0" />
             <dynamics damping="0.0" friction="0.0" />
         </joint>
-        <gazebo reference="gimbal_link_4">
+        <gazebo reference="${namespace}/gimbal_link_4">
           <collision>
             <surface>
@@ -455,5 +446,5 @@
           </collision>
         </gazebo>
-        <link name="gimbal_link_4">
+        <link name="${namespace}/gimbal_link_4">
             <inertial>
                 <mass value="0.0001" />
@@ -461,24 +452,18 @@
                 <inertia ixx="0.0001" ixy="0" ixz="0" iyy="0.0001" iyz="0" izz="0.0001" />
             </inertial>
-<!--             <visual>
-                <geometry>
-                <box size="0.01 0.01 0.01" />
-                </geometry>
-            </visual> -->
             <visual>
               <origin xyz="0 0 0" rpy="0 1.57 0"/>
               <geometry>
-                <!--box size="${camera_link} ${camera_link} ${camera_link}"/-->
                 <mesh filename="package://ardupilot_gazebo/models/util/asus_xtion_pro_camera.dae" scale="1 1 1" />
               </geometry>
             </visual>
         </link>
-        <joint name="camera_gimbal_joint" type="continuous">
-            <parent link="gimbal_link_4" />
-            <child link="camera_link" />
+        <joint name="${namespace}/camera_gimbal_joint" type="continuous">
+            <parent link="${namespace}/gimbal_link_4" />
+            <child link="${namespace}/camera_link" />
             <axis xyz="0 0 1" />
             <dynamics damping="0.0" friction="0.0" />
         </joint>
-        <gazebo reference="camera_link">
+        <gazebo reference="${namespace}/camera_link">
           <collision>
             <surface>
@@ -489,15 +474,15 @@
           </collision>
         </gazebo>
-        <link name="camera_link">
+        <link name="${namespace}/camera_link">
         </link>
-        <joint name="camera_optical_joint" type="fixed">
+        <joint name="${namespace}/camera_optical_joint" type="fixed">
             <origin xyz="0 0 0" rpy="${-pi/2} 0.0 ${-pi/2}" />
-            <parent link="camera_link" />
-            <child link="camera_optical_frame"/>
+            <parent link="${namespace}/camera_link" />
+            <child link="${namespace}/camera_optical_frame"/>
         </joint>
-        <gazebo reference="camera_optical_joint">
+        <gazebo reference="${namespace}/camera_optical_joint">
             <preserveFixedJoint>true</preserveFixedJoint>
         </gazebo>
-        <gazebo reference="camera_optical_frame">
+        <gazebo reference="${namespace}/camera_optical_frame">
           <collision>
             <surface>
@@ -508,7 +493,7 @@
           </collision>
         </gazebo>
-        <link name="camera_optical_frame">
+        <link name="${namespace}/camera_optical_frame">
         </link>
-        <gazebo reference="gimbal_link_4">
+        <gazebo reference="${namespace}/gimbal_link_4">
             <sensor type="depth" name="camera">
               <update_rate>50.0</update_rate>
@@ -536,11 +521,11 @@
                   will control the frame rate. -->
                 <updateRate>0.0</updateRate>
-                <cameraName>${namespace}/camera_ir</cameraName>
-                <imageTopicName>/${namespace}/camera/color/image_raw</imageTopicName>
-                <cameraInfoTopicName>/${namespace}/camera/color/camera_info</cameraInfoTopicName>
-                <depthImageTopicName>/${namespace}/camera/depth/image_raw</depthImageTopicName>
-                <depthImageCameraInfoTopicName>/${namespace}/camera/depth/camera_info</depthImageCameraInfoTopicName>
-                <pointCloudTopicName>/${namespace}/camera/depth/points</pointCloudTopicName>
-                <frameName>camera_optical_frame</frameName>
+                <cameraName>${namespace}/camera_ir_gimbal</cameraName>
+                <imageTopicName>/${namespace}/camera_gimbal/color/image_raw</imageTopicName>
+                <cameraInfoTopicName>/${namespace}/camera_gimbal/color/camera_info</cameraInfoTopicName>
+                <depthImageTopicName>/${namespace}/camera_gimbal/depth/image_raw</depthImageTopicName>
+                <depthImageCameraInfoTopicName>/${namespace}/camera_gimbal/depth/camera_info</depthImageCameraInfoTopicName>
+                <pointCloudTopicName>/${namespace}/camera_gimbal/depth/points</pointCloudTopicName>
+                <frameName>camera_gimbal_optical_frame</frameName>
                 <pointCloudCutoff>2.0</pointCloudCutoff>
                 <pointCloudCutoffMax>15.0</pointCloudCutoffMax>
@@ -559,17 +544,19 @@
         </gazebo>
         <gazebo>
-          <plugin name="gimbal_controller" filename="libGazeboGimbalPlugin.so"/>
+          <plugin name="gimbal_controller" filename="libGazeboGimbalPlugin.so">
+            <namespace>${namespace}</namespace>
+          </plugin>
         </gazebo>
         <xacro:transmisija
           trans_number="g1"
-          joint_name="gimbal_roll_joint">
+          joint_name="${namespace}/gimbal_roll_joint">
         </xacro:transmisija>
         <xacro:transmisija
           trans_number="g2"
-          joint_name="gimbal_pitch_joint">
+          joint_name="${namespace}/gimbal_pitch_joint">
         </xacro:transmisija>
         <xacro:transmisija
           trans_number="g3"
-          joint_name="gimbal_yaw_joint">
+          joint_name="${namespace}/gimbal_yaw_joint">
         </xacro:transmisija>
     </xacro:macro>

Commit message: Update motor parameters - kopterworx(big)

File: models/kopterworx/urdf/kopterworx.urdf.xacro (robot description, xacro)
@@ -53,5 +53,5 @@
     rotor_2_joint="${namespace}::${namespace}/rotor_2_joint"
     rotor_3_joint="${namespace}::${namespace}/rotor_3_joint"
-    thrust_multiplier="600"
+    thrust_multiplier="667"
     fdm_port_in="${fdm_port_in}"
     fdm_port_out="${fdm_port_out}">

File: models/kopterworx/urdf/kopterworx_base.urdf.xacro (robot description, xacro)
@@ -8,5 +8,5 @@
   <xacro:property name="mesh_file" value="ardupilot_gazebo/models/kopterworx/meshes/kopterworx_model_simple.dae" />
   <xacro:property name="mesh_scale" value="0.1" />
-  <xacro:property name="prop_scale" value="0.002" />
+  <xacro:property name="prop_scale" value="0.003" />
   <xacro:property name="mass" value="9" />  <!-- [kg] -->
   <xacro:property name="body_width" value="0.3" /> <!-- [m] -->
@@ -19,9 +19,9 @@
   <xacro:property name="mass_rotor" value="0.01" /> <!-- [kg] -->
   <xacro:property name="radius_rotor" value="0.285" /> <!-- [m] -->
-  <xacro:property name="motor_constant" value="0.000285576174524687" /> <!-- [kg*m/s^2] -->
-  <xacro:property name="moment_constant" value="0.041365783102071" /> <!-- [m] -->
+  <xacro:property name="motor_constant" value="2.440724623743665e-04" /> <!-- [kg*m/s^2] -->
+  <xacro:property name="moment_constant" value="0.044148079282817" /> <!-- [m] -->
   <xacro:property name="time_constant_up" value="0.0125" /> <!-- [s] -->
   <xacro:property name="time_constant_down" value="0.0125" /> <!-- [s] -->
-  <xacro:property name="max_rot_velocity" value="600" /> <!-- [rad/s] -->
+  <xacro:property name="max_rot_velocity" value="667" /> <!-- [rad/s] -->
   <xacro:property name="rotor_drag_coefficient" value="8.06428e-05" />
   <xacro:property name="rolling_moment_coefficient" value="0.000001" />
