Commit message: [kopterworx.launch] add enable_tilt_rotors flag

File: models/kopterworx/urdf/kopterworx.urdf.xacro (robot description, xacro)
@@ -6,4 +6,5 @@
   <xacro:property name="enable_gimbal" value="$(arg enable_gimbal)"/>
   <xacro:property name="enable_rotating_velodyne" value="$(arg enable_rotating_velodyne)" />
+  <xacro:property name="enable_tilt_rotors" value="$(arg enable_tilt_rotors)"/>
   <xacro:property name="fdm_port_in" value="$(arg fdm_port_in)"/>
   <xacro:property name="fdm_port_out" value="$(arg fdm_port_out)"/>
@@ -39,5 +40,12 @@
   </xacro:property>
   <!-- Instantiate kopterworx mechanics "mechanics" -->
-  <xacro:include filename="$(find ardupilot_gazebo)/models/kopterworx/urdf/kopterworx_base.urdf.xacro" />
+  <!-- Setup regular quadrotor -->
+  <xacro:unless value="${enable_tilt_rotors}">
+    <xacro:include filename="$(find ardupilot_gazebo)/models/kopterworx/urdf/kopterworx_base.urdf.xacro" />
+  </xacro:unless>
+  <!-- Setup tilt quadrotor -->
+  <xacro:if value="${enable_tilt_rotors}">
+    <xacro:include filename="$(find ardupilot_gazebo)/models/kopterworx/urdf/kopterworx_tilt_base.urdf.xacro" />
+  </xacro:if>
   <xacro:include filename="$(find rotors_description)/urdf/component_snippets.xacro" />
   <!-- Ardupilot plugin

File: models/kopterworx/urdf/kopterworx_tilt_base.urdf.xacro (robot description, xacro)
@@ -19,9 +19,9 @@
   <xacro:property name="mass_rotor" value="0.01" /> <!-- [kg] -->
   <xacro:property name="radius_rotor" value="0.285" /> <!-- [m] -->
-  <xacro:property name="motor_constant" value="0.000285576174524687" /> <!-- [kg*m/s^2] -->
-  <xacro:property name="moment_constant" value="0.041365783102071" /> <!-- [m] -->
+  <xacro:property name="motor_constant" value="2.440724623743665e-04" /> <!-- [kg*m/s^2] -->
+  <xacro:property name="moment_constant" value="0.044148079282817" /> <!-- [m] -->
   <xacro:property name="time_constant_up" value="0.0125" /> <!-- [s] -->
   <xacro:property name="time_constant_down" value="0.0125" /> <!-- [s] -->
-  <xacro:property name="max_rot_velocity" value="600" /> <!-- [rad/s] -->
+  <xacro:property name="max_rot_velocity" value="667" /> <!-- [rad/s] -->
   <xacro:property name="rotor_drag_coefficient" value="8.06428e-05" />
   <xacro:property name="rolling_moment_coefficient" value="0.000001" />
@@ -34,4 +34,7 @@
   <xacro:property name="tilt_z_offset" value="0.1" />
   <xacro:property name="prop_z_offset" value="${tilt_length}" />
+  <!-- Collision bitmask - By default collides with everything -->
+  <xacro:arg name="collision_bitmask" default="-1" />
+  <xacro:property name="collision_bitmask" value="$(arg collision_bitmask)" />
   <!-- Property Blocks -->
   <xacro:property name="body_inertia">
@@ -199,98 +202,4 @@
     <xacro:insert_block name="rotor_inertia" />
   </xacro:vertical_rotor>
-  <!-- Instantiate manipulator center of mass -->
-  <xacro:movable_mass_linear
-    robot_namespace="$(arg namespace)"
-    number="0"
-    parent="$(arg namespace)/base_link"
-    mass="0.5"
-    radius="0.05"
-    limit_low="-0.2"
-    limit_high="0.2"
-    color="Yellow"
-    x_axis="1"
-    y_axis="0"
-    z_axis="0">
-    <origin xyz="0 0 -0.15" rpy="0 0 0" />
-  </xacro:movable_mass_linear>
-  <!-- Instantiate manipulator center of mass transmission -->
-  <xacro:movable_mass_pos_transmission
-    number="0"
-    joint_name="red/movable_mass_joint_0">
-  </xacro:movable_mass_pos_transmission>
-  <!-- Instantiate movable masses -->
-  <xacro:movable_mass_linear
-    robot_namespace="$(arg namespace)"
-    number="1"
-    parent="$(arg namespace)/base_link"
-    mass="0.25"
-    radius="0.03"
-    limit_low="0.2"
-    limit_high="0.5"
-    color="Orange"
-    x_axis="${sin45}"
-    y_axis="${-sin45}"
-    z_axis="0">
-    <origin xyz="0 0 0" rpy="0 0 0" />
-  </xacro:movable_mass_linear>
-  <xacro:movable_mass_linear
-    robot_namespace="$(arg namespace)"
-    number="2"
-    parent="$(arg namespace)/base_link"
-    mass="0.25"
-    radius="0.03"
-    limit_low="0.2"
-    limit_high="0.5"
-    color="Orange"
-    x_axis="${sin45}"
-    y_axis="${sin45}"
-    z_axis="0">
-    <origin xyz="0 0 0" rpy="0 0 0" />
-  </xacro:movable_mass_linear>
-  <xacro:movable_mass_linear
-    robot_namespace="$(arg namespace)"
-    number="3"
-    parent="$(arg namespace)/base_link"
-    mass="0.25"
-    radius="0.03"
-    limit_low="0.2"
-    limit_high="0.5"
-    color="Orange"
-    x_axis="${-sin45}"
-    y_axis="${sin45}"
-    z_axis="0">
-    <origin xyz="0 0 0" rpy="0 0 0" />
-  </xacro:movable_mass_linear>
-  <xacro:movable_mass_linear
-    robot_namespace="$(arg namespace)"
-    number="4"
-    parent="$(arg namespace)/base_link"
-    mass="0.25"
-    radius="0.03"
-    limit_low="0.2"
-    limit_high="0.5"
-    color="Orange"
-    x_axis="${-sin45}"
-    y_axis="${-sin45}"
-    z_axis="0">
-    <origin xyz="0 0 0" rpy="0 0 0" />
-  </xacro:movable_mass_linear>
-  <!-- Instantiate movable masses transmissions -->
-  <xacro:movable_mass_vel_transmission
-    number="1"
-    joint_name="red/movable_mass_joint_1">
-  </xacro:movable_mass_vel_transmission>
-  <xacro:movable_mass_vel_transmission
-    number="2"
-    joint_name="red/movable_mass_joint_2">
-  </xacro:movable_mass_vel_transmission>
-  <xacro:movable_mass_vel_transmission
-    number="3"
-    joint_name="red/movable_mass_joint_3">
-  </xacro:movable_mass_vel_transmission>
-  <xacro:movable_mass_vel_transmission
-    number="4"
-    joint_name="red/movable_mass_joint_4">
-  </xacro:movable_mass_vel_transmission>
   <gazebo reference="$(arg namespace)/base_link">
     <dampingFactor>0.001</dampingFactor>

Commit message: [kopterworx] Add enable_simple_manipulator flag

File: models/kopterworx/urdf/kopterworx.urdf.xacro (robot description, xacro)
@@ -7,4 +7,5 @@
   <xacro:property name="enable_rotating_velodyne" value="$(arg enable_rotating_velodyne)" />
   <xacro:property name="enable_tilt_rotors" value="$(arg enable_tilt_rotors)"/>
+  <xacro:property name="enable_simple_manipulator" value="$(arg enable_simple_manipulator)"/>
   <xacro:property name="fdm_port_in" value="$(arg fdm_port_in)"/>
   <xacro:property name="fdm_port_out" value="$(arg fdm_port_out)"/>
@@ -47,4 +48,32 @@
   <xacro:if value="${enable_tilt_rotors}">
     <xacro:include filename="$(find ardupilot_gazebo)/models/kopterworx/urdf/kopterworx_tilt_base.urdf.xacro" />
+  </xacro:if>
+  <xacro:if value="${enable_simple_manipulator}">
+    <xacro:include filename="$(find ardupilot_gazebo)/models/util/multirotor_movable_masses.urdf.xacro"/>
+    <!-- Instantiate manipulator center of mass -->
+    <xacro:simple_manipulator
+      robot_namespace="$(arg namespace)"
+      number="0"
+      parent="$(arg namespace)/base_link"
+      mass="1.0"
+      radius="0.05"
+      limit_low="-0.5"
+      limit_high="0.5"
+      color="Yellow">
+      <origin xyz="0 0 -0.125" rpy="0 0 0" />
+    </xacro:simple_manipulator>
+    <!-- Instantiate manipulator center of mass transmission -->
+    <xacro:movable_mass_pos_transmission
+      number="0"
+      joint_name="red/movable_mass_x_joint_0">
+    </xacro:movable_mass_pos_transmission>
+    <xacro:movable_mass_pos_transmission
+      number="1"
+      joint_name="red/movable_mass_y_joint_0">
+    </xacro:movable_mass_pos_transmission>
+    <xacro:movable_mass_pos_transmission
+      number="2"
+      joint_name="red/movable_mass_z_joint_0">
+    </xacro:movable_mass_pos_transmission>
   </xacro:if>
   <xacro:include filename="$(find rotors_description)/urdf/component_snippets.xacro" />

File: models/util/multirotor_tilt.urdf.xacro (robot description, xacro)
@@ -28,34 +28,4 @@
     </link>
   </xacro:macro>
-  <!-- Macro for movable mass on a straight line. -->
-  <xacro:macro name="movable_mass_linear"
-    params="robot_namespace number parent mass radius limit_low limit_high color x_axis y_axis z_axis *origin">
-    <joint name="${robot_namespace}/movable_mass_joint_${number}" type="prismatic">
-      <xacro:insert_block name="origin"/>
-      <axis xyz="${x_axis} ${y_axis} ${z_axis}"/>
-      <parent link="${parent}"/>
-      <child link="${robot_namespace}/movable_mass_link_${number}"/>
-      <limit lower="${limit_low}" upper="${limit_high}" effort="10000" velocity="20"/>
-    </joint>
-    <link name="${robot_namespace}/movable_mass_link_${number}">
-      <visual>
-        <origin rpy="0 0 0" xyz="0 0 0"/>
-        <geometry>
-          <sphere radius="${radius}"/>
-        </geometry>
-      </visual>
-      <inertial>
-        <origin rpy="0 0 0" xyz="0 0 0"/>
-        <mass value="${mass}"/>
-        <inertia
-            ixx="${2/5 * mass * radius * radius}"     ixy="0.0"                                  ixz="0.0"
-            iyx="0.0"                                 iyy="${2/5 * mass * radius * radius}"      iyz="0.0"
-            izx="0.0"                                 izy="0.0"                                  izz="${2/5 * mass * radius * radius}" />
-      </inertial>
-    </link>
-    <gazebo reference="${robot_namespace}/movable_mass_link_${number}">
-      <material>Gazebo/${color}</material>
-    </gazebo>
-  </xacro:macro>
   <!-- We add a <transmission> block for every joint that we wish to actuate. -->
   <xacro:macro name="tilt_joint_transmission" params="number joint_name">
@@ -70,25 +40,3 @@
     </transmission>
   </xacro:macro>
-  <xacro:macro name="movable_mass_pos_transmission" params="number joint_name">
-    <transmission name="movable_mass_pos_transmission_${number}">
-      <type>transmission_interface/SimpleTransmission</type>
-      <actuator name="movable_mass_motor_${number}">
-        <mechanicalReduction>1</mechanicalReduction>
-      </actuator>
-      <joint name="${joint_name}">
-        <hardwareInterface>hardware_interface/PositionJointInterface</hardwareInterface>
-      </joint>
-    </transmission>
-  </xacro:macro>
-  <xacro:macro name="movable_mass_vel_transmission" params="number joint_name">
-    <transmission name="movable_mass_vel_transmission_${number}">
-      <type>transmission_interface/SimpleTransmission</type>
-      <actuator name="movable_mass_motor_${number}">
-        <mechanicalReduction>1</mechanicalReduction>
-      </actuator>
-      <joint name="${joint_name}">
-        <hardwareInterface>hardware_interface/VelocityJointInterface</hardwareInterface>
-      </joint>
-    </transmission>
-  </xacro:macro>
 </robot>
