Commit message: Add fdm_ports as parameters to ardupilot macro.

File: models/ardrone/urdf/uav.gazebo.xacro (robot description, xacro)
@@ -115,5 +115,7 @@
 		rotor_2_joint="uav::rotor_2_joint"
 		rotor_3_joint="uav::rotor_3_joint"
-		thrust_multiplier="1475">
+		thrust_multiplier="1475"
+    fdm_port_in="9002"
+		fdm_port_out="9003">
 	</xacro:ardupilot>
 </robot>

File: models/bebop/urdf/bebop.urdf.xacro (robot description, xacro)
@@ -75,5 +75,7 @@
 		rotor_2_joint="bebop::rotor_2_joint"
 		rotor_3_joint="bebop::rotor_3_joint"
-		thrust_multiplier="1000">
+		thrust_multiplier="1000"
+		fdm_port_in="9002"
+		fdm_port_out="9003">
 	</xacro:ardupilot>
     <link name="laser1D_link">

File: models/kopterworx/urdf/kopterworx.urdf.xacro (robot description, xacro)
@@ -3,4 +3,6 @@
   <xacro:property name="namespace" value="$(arg namespace)" />
   <xacro:property name="enable_velodyne" value="$(arg enable_velodyne)"/>
+	<xacro:property name="fdm_port_in" value="$(arg fdm_port_in)"/>
+	<xacro:property name="fdm_port_out" value="$(arg fdm_port_out)"/>
 	<xacro:property name="horizontal_velodyne_origin">
     <origin xyz="0.08 0. -0.1578" rpy="3.141592653589793 0.1323284641020683 0." />
@@ -33,5 +35,7 @@
 		rotor_2_joint="${namespace}::rotor_2_joint"
 		rotor_3_joint="${namespace}::rotor_3_joint"
-		thrust_multiplier="600">
+		thrust_multiplier="600"
+		fdm_port_in="${fdm_port_in}"
+		fdm_port_out="${fdm_port_out}">
 	</xacro:ardupilot>
 	<xacro:if value="${enable_velodyne}">

File: models/util/multirotor_base.urdf.xacro (robot description, xacro)
@@ -146,5 +146,5 @@
   <!-- TODO(lmark): Ardupilot macro cleanup -->
   <xacro:macro name="ardupilot"
-    params="imu_topic control_topic imu_sensor_name rotor_0_joint rotor_1_joint rotor_2_joint rotor_3_joint thrust_multiplier">
+    params="imu_topic control_topic imu_sensor_name rotor_0_joint rotor_1_joint rotor_2_joint rotor_3_joint thrust_multiplier fdm_port_in fdm_port_out">
      <gazebo>
         <plugin name="arducopter_plugin" filename="libArduPilotPlugin.so">
@@ -152,6 +152,6 @@
         <controlTopicName>${control_topic}</controlTopicName>
         <fdm_addr>127.0.0.1</fdm_addr>
-        <fdm_port_in>9002</fdm_port_in>
-        <fdm_port_out>9003</fdm_port_out>
+        <fdm_port_in>${fdm_port_in}</fdm_port_in>
+        <fdm_port_out>${fdm_port_out}</fdm_port_out>
         <!--
             Require by APM :
