Commit message: Ardudrone model in SITL.

File: models/ardrone/urdf/uav.base.urdf.xacro (robot description, xacro)
@@ -85,5 +85,5 @@
     robot_namespace="$(arg name)"
     suffix="front_left"
-    direction="cw"
+    direction="ccw"
     motor_constant="${motor_constant}"
     moment_constant="${moment_constant}"
@@ -105,5 +105,5 @@
     robot_namespace="$(arg name)"
     suffix="front_right"
-    direction="ccw"
+    direction="cw"
     motor_constant="${motor_constant}"
     moment_constant="${moment_constant}"
@@ -125,5 +125,5 @@
     robot_namespace="$(arg name)"
     suffix="back_left"
-    direction="ccw"
+    direction="cw"
     motor_constant="${motor_constant}"
     moment_constant="${moment_constant}"
@@ -145,5 +145,5 @@
     robot_namespace="$(arg name)"
     suffix="back_right"
-    direction="cw"
+    direction="ccw"
     motor_constant="${motor_constant}"
     moment_constant="${moment_constant}"

File: models/ardrone/urdf/uav.gazebo.xacro (robot description, xacro)
@@ -37,28 +37,4 @@
     <limit upper="0" lower="0" effort="0" velocity="0" />
   </joint>
-  <!-- Mount an IMU -->
-  <gazebo>
-    <!-- IMU -->
-    <plugin filename="libhector_gazebo_ros_imu.so" name="imu_ros">
-      <!-- parameters according to http://wiki.ros.org/hector_gazebo_plugins#GazeboRosImu -->
-      <!-- robotNamespace>${namespace}</robotNamespace -->
-      <robotNamespace>$(arg name)</robotNamespace>
-      <bodyName>imu_link</bodyName> <!-- (string, required): name of the body which holds the IMU sensor -->
-      <topicName>imu</topicName> <!-- (string): name of the sensor output topic and prefix of service names (defaults to imu) -->
-      <accelOffset>0.0 0.0 0.0</accelOffset> <!-- (Vector3): constant acceleration offset -->
-      <accelDrift>0.0 0.0 0.0</accelDrift> <!-- (Vector3): standard deviation of the acceleration drift error -->
-      <accelDriftFrequency>0.0 0.0 0.0</accelDriftFrequency> <!-- (Vector3): mean frequency of the acceleration drift staviti na nulu-->
-      <accelGaussianNoise>0.001 0.001 0.001</accelGaussianNoise> <!-- (Vector3): standard deviation of the additive Gaussian acceleration noise -->
-      <rateOffset>0.0 0.0 0.0</rateOffset> <!-- (Vector3): constant rate offset -->
-      <rateDrift>0.0 0.0 0.0</rateDrift> <!-- (Vector3): standard deviation of the rate drift error -->
-      <rateDriftFrequency>0.0 0.0 0.0</rateDriftFrequency> <!-- (Vector3): mean frequency of the rate drift  staviti na nulu-->
-      <rateGaussianNoise>0.0001 0.0001 0.0001</rateGaussianNoise> <!-- (Vector3): standard deviation of the additive Gaussian rate noise -->
-      <headingOffset>0.0</headingOffset> <!-- (double): constant heading offset -->
-      <headingDrift>0.0</headingDrift> <!-- (double): standard deviation of the heading drift error -->
-      <headingDriftFrequency>0.0</headingDriftFrequency> <!-- (double): mean frequency of the heading drift  staviti na nulu-->
-      <headingGaussianNoise>0.0</headingGaussianNoise> <!-- (double): standard deviation of the heading additive Gaussian noise -->
-      <rpyOffsets>0.0 0.0 0.0</rpyOffsets> <!-- (Vector3): if non-zero, used to calculate accelOffset and headingOffset so that resulting roll, pitch and yaw errors correspond to this values when the platform is leveled (for compatibility with gazebo_plugins) -->
-    </plugin>
-  </gazebo>
   <xacro:if value="${mount_magnet}">
     <xacro:if value="${mount_magnet_with_disk}">
@@ -139,5 +115,5 @@
 		rotor_2_joint="uav::rotor_2_joint"
 		rotor_3_joint="uav::rotor_3_joint"
-		thrust_multiplier="1000">
+		thrust_multiplier="1475">
 	</xacro:ardupilot>
 </robot>

File: models/util/multirotor_base.urdf.xacro (robot description, xacro)
@@ -7,5 +7,4 @@
     <joint name="base_joint" type="fixed">
       <xacro:insert_block name="origin"/>
-      <origin xyz="0 0 0" rpy="0 0 0" />
       <parent link="base_link" />
       <child link="base_link_inertia" />
@@ -18,5 +17,4 @@
       </inertial>
       <visual>
-        <origin xyz="0 0 0" rpy="0 0 0" />
         <geometry>
           <mesh filename="package://${mesh_file}"
@@ -26,8 +24,8 @@
       </visual>
       <collision>
-        <origin xyz="0 0 0.0" rpy="0 0 0" />
         <geometry>
           <mesh filename="package://${mesh_file}"
             scale="${mesh_scale} ${mesh_scale} ${mesh_scale}" /> <!-- [m] [m] [m] -->
+          <!-- box size="${body_width} ${body_width} ${body_height}"/ --> <!-- [m] [m] [m] -->
         </geometry>
       </collision>
@@ -64,5 +62,4 @@
     <!-- IMU joint -->
     <joint name="imu_joint" type="revolute">
-      <!--origin xyz="0 0 0" rpy="3.1416 0 0" / -->
       <parent link="base_link" />
       <child link="imu_link" />
@@ -162,5 +159,5 @@
           <jointName>${rotor_1_joint}</jointName>
           <multiplier>${thrust_multiplier}</multiplier>
-          <controlVelocitySlowdownSim>30</controlVelocitySlowdownSim>
+          <controlVelocitySlowdownSim>15</controlVelocitySlowdownSim>
         </control>
         <control channel="1">
@@ -169,5 +166,5 @@
           <jointName>${rotor_3_joint}</jointName>
           <multiplier>${thrust_multiplier}</multiplier>
-          <controlVelocitySlowdownSim>30</controlVelocitySlowdownSim>
+          <controlVelocitySlowdownSim>15</controlVelocitySlowdownSim>
         </control>
         <control channel="2">
@@ -175,6 +172,6 @@
           <offset>0</offset>
           <jointName>${rotor_0_joint}</jointName>
-          <multiplier>-${thrust_multiplier}</multiplier>
-          <controlVelocitySlowdownSim>30</controlVelocitySlowdownSim>
+          <multiplier>${thrust_multiplier}</multiplier>
+          <controlVelocitySlowdownSim>15</controlVelocitySlowdownSim>
         </control>
         <control channel="3">
@@ -182,6 +179,6 @@
           <offset>0</offset>
           <jointName>${rotor_2_joint}</jointName>
-          <multiplier>-${thrust_multiplier}</multiplier>
-          <controlVelocitySlowdownSim>30</controlVelocitySlowdownSim>
+          <multiplier>${thrust_multiplier}</multiplier>
+          <controlVelocitySlowdownSim>15</controlVelocitySlowdownSim>
         </control>
       </plugin>

Commit message: [arducopter] Accomodate URDF files.

File: models/ardrone/urdf/uav.base.urdf.xacro (robot description, xacro)
@@ -10,4 +10,5 @@
   <xacro:property name="mesh_file" value="ardupilot_gazebo/models/ardrone/meshes/3DR_Arducopter.dae" />
   <xacro:property name="mesh_scale" value="1" />
+  <xacro:property name="prop_scale" value="0.001" />
   <xacro:property name="mass" value="2.083" />  <!-- [kg] -->
   <xacro:property name="body_width" value="0.1" /> <!-- [m] -->
@@ -97,5 +98,6 @@
     rotor_drag_coefficient="${rotor_drag_coefficient}"
     rolling_moment_coefficient="${rolling_moment_coefficient}"
-    color="Blue">
+    color="Blue"
+    prop_scale="${prop_scale}">
     <!--<origin xyz="${cos45*arm_length} ${sin45*arm_length} ${rotor_offset_top}" rpy="0 0 0" />-->
     <origin xyz="${1*arm_length} ${0*arm_length} ${rotor_offset_top}" rpy="0 ${-tilt_angle} 0" />
@@ -117,5 +119,6 @@
     rotor_drag_coefficient="${rotor_drag_coefficient}"
     rolling_moment_coefficient="${rolling_moment_coefficient}"
-    color="Red">
+    color="Red"
+    prop_scale="${prop_scale}">
     <!--<origin xyz="${cos45*arm_length} ${-sin45*arm_length} ${rotor_offset_top}" rpy="0 0 0" />-->
     <origin xyz="${0*arm_length} ${-1*arm_length} ${rotor_offset_top}" rpy="${-tilt_angle} 0 0" />
@@ -137,5 +140,6 @@
     rotor_drag_coefficient="${rotor_drag_coefficient}"
     rolling_moment_coefficient="${rolling_moment_coefficient}"
-    color="Red">
+    color="Red"
+    prop_scale="${prop_scale}">
     <!--<origin xyz="${-cos45*arm_length} ${sin45*arm_length} ${rotor_offset_top}" rpy="0 0 0" />-->
     <origin xyz="${0*arm_length} ${1*arm_length} ${rotor_offset_top}" rpy="${tilt_angle} 0 0" />
@@ -157,5 +161,6 @@
     rotor_drag_coefficient="${rotor_drag_coefficient}"
     rolling_moment_coefficient="${rolling_moment_coefficient}"
-    color="Blue">
+    color="Blue"
+    prop_scale="${prop_scale}">
     <!--<origin xyz="${-cos45*arm_length} ${-sin45*arm_length} ${rotor_offset_top}" rpy="0 0 0" />-->
     <origin xyz="${-1*arm_length} ${0*arm_length} ${rotor_offset_top}" rpy="0 ${tilt_angle} 0" />

File: models/ardrone/urdf/uav.gazebo.xacro (robot description, xacro)
@@ -108,6 +108,6 @@
   </xacro:odometry_plugin_macro>
 	<xacro:ardupilot
-		imu_topic="/uav/imu"
-		control_topic="/gazebo/command/motor_speed"
+		imu_topic="/$(arg name)/imu"
+		control_topic="/$(arg name)/gazebo/command/motor_speed"
 		imu_sensor_name="uav::imu_link::imu_sensor"
 		rotor_0_joint="uav::rotor_0_joint"
