Commit message: Initial Kopterworx model structure.

File: models/util/multirotor_base.urdf.xacro (robot description, xacro)
@@ -1,4 +1,18 @@
 <?xml version="1.0"?>
 <robot xmlns:xacro="http://ros.org/wiki/xacro">
+  <!-- Macro for the inertia of a box -->
+  <xacro:macro name="box_inertia" params="x y z mass">
+    <inertia ixx="${0.0833333 * mass * (y*y + z*z)}" ixy="0.0" ixz="0.0"
+      iyy="${0.0833333 * mass * (x*x + z*z)}" iyz="0.0"
+      izz="${0.0833333 * mass * (x*x + y*y)}" />
+  </xacro:macro>
+  <!-- Macro for the inertial properties of a box -->
+  <xacro:macro name="box_inertial" params="x y z mass *origin">
+    <inertial>
+      <mass value="${mass}" />
+      <xacro:insert_block name="origin" />
+      <xacro:box_inertia x="${x}" y="${y}" z="${z}" mass="${mass}" />
+    </inertial>
+  </xacro:macro>
   <!-- Main multirotor link -->
   <xacro:macro name="multirotor_base_macro"
@@ -18,14 +32,14 @@
       <visual>
         <geometry>
-          <mesh filename="package://${mesh_file}"
-            scale="${mesh_scale} ${mesh_scale} ${mesh_scale}" />
-          <!-- box size="${body_width} ${body_width} ${body_height}"/ --> <!-- [m] [m] [m] -->
+          <!-- mesh filename="package://${mesh_file}"
+            scale="${mesh_scale} ${mesh_scale} ${mesh_scale}" /-->
+          <box size="${body_width} ${body_width} ${body_height}"/> <!-- [m] [m] [m] -->
         </geometry>
       </visual>
       <collision>
         <geometry>
-          <mesh filename="package://${mesh_file}"
-            scale="${mesh_scale} ${mesh_scale} ${mesh_scale}" /> <!-- [m] [m] [m] -->
-          <!-- box size="${body_width} ${body_width} ${body_height}"/ --> <!-- [m] [m] [m] -->
+          <!-- mesh filename="package://${mesh_file}"
+            scale="${mesh_scale} ${mesh_scale} ${mesh_scale}" /--> <!-- [m] [m] [m] -->
+          <box size="${body_width} ${body_width} ${body_height}"/> <!-- [m] [m] [m] -->
         </geometry>
       </collision>

Commit message: [multirotor_base.urdf] Mesh - visual and box - collision in multirotor_base_macro

File: models/util/multirotor_base.urdf.xacro (robot description, xacro)
@@ -32,7 +32,7 @@
       <visual>
         <geometry>
-          <!-- mesh filename="package://${mesh_file}"
-            scale="${mesh_scale} ${mesh_scale} ${mesh_scale}" /-->
-          <box size="${body_width} ${body_width} ${body_height}"/> <!-- [m] [m] [m] -->
+          <mesh filename="package://${mesh_file}"
+            scale="${mesh_scale} ${mesh_scale} ${mesh_scale}" />
+          <!--box size="${body_width} ${body_width} ${body_height}"/--> <!-- [m] [m] [m] -->
         </geometry>
       </visual>
@@ -91,5 +91,5 @@
   <!-- Rotor joint and link -->
   <xacro:macro name="vertical_rotor"
-    params="robot_namespace suffix direction motor_constant moment_constant parent mass_rotor radius_rotor time_constant_up time_constant_down max_rot_velocity motor_number rotor_drag_coefficient rolling_moment_coefficient color *origin *inertia">
+    params="robot_namespace suffix direction motor_constant moment_constant parent mass_rotor radius_rotor time_constant_up time_constant_down max_rot_velocity motor_number rotor_drag_coefficient rolling_moment_coefficient color prop_scale *origin *inertia">
     <joint name="rotor_${motor_number}_joint" type="continuous">
       <xacro:insert_block name="origin" />
@@ -112,5 +112,5 @@
           <!-- <cylinder length="0.005" radius="${radius_rotor}"/> --> <!-- [m] -->
           <mesh filename="package://ardupilot_gazebo/models/util/propeller_${direction}.dae"
-            scale="0.00055 0.00055 0.00055" />
+            scale="${prop_scale} ${prop_scale} ${prop_scale}" />
           <!-- <box size="${2*radius_rotor} 0.01 0.005"/> -->
         </geometry>

Commit message: [multirotor_base] Now visualise camera mesh.

File: models/util/multirotor_base.urdf.xacro (robot description, xacro)
@@ -217,11 +217,11 @@
         </geometry>
       </collision-->
-      <!--visual>
-        <origin xyz="0 0 0" rpy="0 0 0"/>
-        <geometry>
-          <box size="${camera_link} ${camera_link} ${camera_link}"/>
-        </geometry>
-        <material name="red"/>
-      </visual-->
+      <visual>
+        <origin xyz="0 0 0" rpy="0 1.57 0"/>
+        <geometry>
+          <!--box size="${camera_link} ${camera_link} ${camera_link}"/-->
+          <mesh filename="package://ardupilot_gazebo/models/util/asus_xtion_pro_camera.dae" scale="1 1 1" />
+        </geometry>
+      </visual>
       <inertial>
         <mass value="${camera_mass}" />
@@ -265,5 +265,5 @@
           <imageTopicName>/${namespace}/camera/color/image_raw</imageTopicName>
           <cameraInfoTopicName>/${namespace}/camera/color/camera_info</cameraInfoTopicName>
-          <depthImageTopicName>/camera/depth/image_raw</depthImageTopicName>
+          <depthImageTopicName>/${namespace}/camera/depth/image_raw</depthImageTopicName>
           <depthImageCameraInfoTopicName>/${namespace}/camera/depth/camera_info</depthImageCameraInfoTopicName>
           <pointCloudTopicName>/${namespace}/camera/depth_registered/points</pointCloudTopicName>

Commit message: [multirotor_base] Add a correctly rotated camera link

File: models/util/multirotor_base.urdf.xacro (robot description, xacro)
@@ -234,4 +234,10 @@
       <parent link="${parent}"/>
       <child link="camera_box"/>
+    </joint>
+    <link name="camera"/>
+    <joint name="camera_help" type="fixed">
+      <parent link="camera_box"/>
+      <child link="camera"/>
+      <origin rpy="-1.57 0 -1.57"/>
     </joint>
     <!-- camera -->

Commit message: Add camera visualization

File: models/util/multirotor_base.urdf.xacro (robot description, xacro)
@@ -378,4 +378,11 @@
                 </geometry>
             </visual> -->
+            <visual>
+              <origin xyz="0 0 0" rpy="0 1.57 0"/>
+              <geometry>
+                <!--box size="${camera_link} ${camera_link} ${camera_link}"/-->
+                <mesh filename="package://ardupilot_gazebo/models/util/asus_xtion_pro_camera.dae" scale="1 1 1" />
+              </geometry>
+            </visual>
         </link>
         <joint name="camera_gimbal_joint" type="continuous">
