Commit message: [zephyr_delta_wing] Convert model to urdf

File: models/zephyr_delta_wing/urdf/zephyr.urdf.xacro (robot description, xacro)
@@ -1,6 +1,13 @@
 <?xml version="1.0" ?>
 <robot xmlns:xacro="http://ros.org/wiki/xacro" name="zephyr_delta_wing">
-  <xacro:property name="namespace" value="asd"/>
-  <joint name="${namespace}/zephyr_delta_wing/zephyr/imu_joint" type="fixed">
+  <xacro:property name="namespace" value="$(arg namespace)"/>
+  <!-- base_link -> wing -->
+  <joint name="${namespace}/zephyr_delta_wing/zephyr/base_joint" type="fixed">
+    <parent link="${namespace}/zephyr_delta_wing/base_link"/>
+    <child link="${namespace}/zephyr_delta_wing/wing"/>
+    <origin xyz="0 0 0" rpy="0 0 0"/>
+  </joint>
+  <!-- wing -> imu -->
+  <joint name="${namespace}/zephyr_delta_wing/zephyr/imu_joint" type="revolute">
     <parent link="${namespace}/zephyr_delta_wing/wing"/>
     <child link="${namespace}/zephyr_delta_wing/zephyr/imu_link"/>
@@ -8,12 +15,22 @@
     <axis xyz="0 0 1"/>
     <limit lower="0.0" upper="0.0" effort="0.0" velocity="0.0"/>
-  </joint>
-  <joint name="${namespace}/zephyr_delta_wing/propeller_joint" type="fixed">
+    <dynamics damping="1.0"/>
+  </joint>
+  <gazebo reference="${namespace}/zephyr_delta_wing/zephyr/imu_joint">
+    <implicit_spring_damper>1</implicit_spring_damper>
+    <use_parent_model_frame>1</use_parent_model_frame>
+  </gazebo>
+  <!-- wing -> propeller -->
+  <joint name="${namespace}/zephyr_delta_wing/propeller_joint" type="continuous">
     <parent link="${namespace}/zephyr_delta_wing/wing"/>
     <child link="${namespace}/zephyr_delta_wing/propeller"/>
     <origin xyz="0      0.02    0.021" rpy="0      1.57079 0"/>
     <axis xyz="0 -1  0"/>
-    <limit lower="0" upper="0" effort="0" velocity="0"/>
-  </joint>
+    <dynamics damping="0.002"/>
+  </joint>
+  <gazebo reference="${namespace}/zephyr_delta_wing/propeller_joint">
+    <implicit_spring_damper>1</implicit_spring_damper>
+  </gazebo>
+  <!-- wing -> left_flap -->
   <joint name="${namespace}/zephyr_delta_wing/flap_left_joint" type="revolute">
     <parent link="${namespace}/zephyr_delta_wing/wing"/>
@@ -21,6 +38,7 @@
     <origin xyz="0.438   0.141   0.02" rpy="0 0 0"/>
     <axis xyz="1      0.33032 0"/>
-    <limit lower="-0.524" upper="0.524" effort="0.0" velocity="0.0"/>
-  </joint>
+    <limit lower="-0.524" upper="0.524" effort="30" velocity="10.0"/>
+  </joint>
+  <!-- wing -> right_flap -->
   <joint name="${namespace}/zephyr_delta_wing/flap_right_joint" type="revolute">
     <parent link="${namespace}/zephyr_delta_wing/wing"/>
@@ -28,6 +46,18 @@
     <origin xyz="-0.438    0.141    0.02" rpy="0 0 0"/>
     <axis xyz="1      -0.33032  0"/>
-    <limit lower="-0.524" upper="0.524" effort="0.0" velocity="0.0"/>
-  </joint>
+    <limit lower="-0.524" upper="0.524" effort="30" velocity="10.0"/>
+  </joint>
+  <!-- wing -> skid pad -->
+  <joint name="${namespace}/zephyr_delta_wing/skid_pad_joint" type="fixed">
+    <parent link="${namespace}/zephyr_delta_wing/wing"/>
+    <child link="${namespace}/zephyr_delta_wing/skid_pad"/>
+    <origin xyz="0   -0.07 -0.15" rpy="0 0 0"/>
+  </joint>
+  <gazebo reference="${namespace}/zephyr_delta_wing/skid_pad_joint">
+    <use_parent_model_frame>1</use_parent_model_frame>
+  </gazebo>
+  <!-- base_link -->
+  <link name="${namespace}/zephyr_delta_wing/base_link"/>
+  <!-- wing -->
   <link name="${namespace}/zephyr_delta_wing/wing">
     <inertial>
@@ -61,4 +91,5 @@
     </visual>
   </link>
+  <!-- imu -->
   <link name="${namespace}/zephyr_delta_wing/zephyr/imu_link">
     <inertial>
@@ -68,4 +99,12 @@
     </inertial>
   </link>
+  <gazebo reference="${namespace}/zephyr_delta_wing/zephyr/imu_link">
+    <sensor name="imu_sensor" type="imu">
+        <pose>0 0 0 3.141593 0 -1.57079</pose>
+        <always_on>1</always_on>
+        <update_rate>1000.0</update_rate>
+    </sensor>
+  </gazebo>
+  <!-- Propeller -->
   <link name="${namespace}/zephyr_delta_wing/propeller">
     <inertial>
@@ -93,4 +132,5 @@
     </visual>
   </link>
+  <!-- left flap -->
   <link name="${namespace}/zephyr_delta_wing/flap_left">
     <inertial>
@@ -112,4 +152,5 @@
     </visual>
   </link>
+  <!-- right flap -->
   <link name="${namespace}/zephyr_delta_wing/flap_right">
     <inertial>
@@ -131,3 +172,260 @@
     </visual>
   </link>
+  <!-- skid pad - an invisible platform below the plane to help takeoff -->
+  <link name="${namespace}/zephyr_delta_wing/skid_pad">
+    <inertial>
+      <mass value="0.1"/>
+      <origin xyz="0 0 0" rpy="0 0 0"/>
+      <inertia ixx="0.0043137104" ixy="0" ixz="0" iyy="0.00387382402" iyz="0" izz="0.00809845106"/>
+    </inertial>
+    <collision name="zephyr_delta_wing/skid_pad">
+      <origin xyz="0 0 0" rpy="0 0 0"/>
+      <geometry>
+        <box size="2.0 2.0 0.05"/>
+      </geometry>
+    </collision>
+    <!--visual name="skid_pad">
+        <origin xyz="0 0 0" rpy="0 0 0"/>
+        <geometry>
+          <box size="2.0 2.0 0.05"/>
+        </geometry>
+    </visual-->
+  </link>
+  <!-- Add slipage to the skid pad -->
+  <gazebo reference="${namespace}/zephyr_delta_wing/skid_pad">
+    <kp>100000.0</kp>
+    <kd>1</kd>
+    <minDepth>0.01</minDepth>
+    <maxVel>1.0</maxVel>
+    <mu1>0.3</mu1>
+    <mu2>20</mu2>
+    <fdir1>0 1 0</fdir1>
+  </gazebo>
+  <!-- gps (not used in Ardupilot plugin, currently using Gazebo position)-->
+  <gazebo reference="${namespace}/zephyr_delta_wing/wing">
+  <sensor name="${namespace}/gps_sensor" type="gps">
+    <pose>0 0 0  0 0 0</pose>
+    <update_rate>10.0</update_rate>
+    <always_on>true</always_on>
+    <gps>
+      <position_sensing>
+        <horizontal>
+          <noise type="gaussian_quantized">
+            <mean>0</mean>
+            <stddev>1</stddev>
+            <bias_mean>3</bias_mean>
+            <bias_stddev>1</bias_stddev>
+            <precision>0.5</precision>
+          </noise>
+        </horizontal>
+        <vertical>
+          <noise type="gaussian_quantized">
+            <mean>0</mean>
+            <stddev>1</stddev>
+            <bias_mean>3</bias_mean>
+            <bias_stddev>1</bias_stddev>
+            <precision>1.0</precision>
+          </noise>
+        </vertical>
+      </position_sensing>
+      <velocity_sensing>
+        <horizontal>
+          <noise type="gaussian_quantized">
+            <mean>0</mean>
+            <stddev>0.1</stddev>
+            <bias_mean>0.1</bias_mean>
+            <bias_stddev>0.1</bias_stddev>
+            <precision>0.1</precision>
+          </noise>
+        </horizontal>
+        <vertical>
+          <noise type="gaussian_quantized">
+            <mean>0</mean>
+            <stddev>0.2</stddev>
+            <bias_mean>0.2</bias_mean>
+            <bias_stddev>0.2</bias_stddev>
+            <precision>0.2</precision>
+          </noise>
+        </vertical>
+      </velocity_sensing>
+    </gps>
+  </sensor>
+  </gazebo>
+  <gazebo>
+  <plugin name="invisible_canard" filename="libLiftDragPlugin.so">
+      <a0>0.13</a0>
+      <cla>3.7</cla>
+      <cda>0.06417112299</cda>
+      <cma>-1.8</cma>
+      <alpha_stall>0.3391428111</alpha_stall>
+      <cla_stall>-3.85</cla_stall>
+      <cda_stall>-0.9233984055</cda_stall>
+      <cma_stall>0</cma_stall>
+      <cp>0 -0.1 0</cp>
+      <area>0.50</area>
+      <air_density>1.2041</air_density>
+      <forward>0 -1 0</forward>
+      <upward>0 0 1</upward>
+      <link_name>${namespace}/zephyr_delta_wing/base_link</link_name>
+  </plugin>
+  <plugin name="left_wing" filename="libLiftDragPlugin.so">
+      <a0>0.15</a0>
+      <cla>6.8</cla>
+      <cda>0.06417112299</cda>
+      <cma>-1.8</cma>
+      <alpha_stall>0.6391428111</alpha_stall>
+      <cla_stall>-3.85</cla_stall>
+      <cda_stall>-0.9233984055</cda_stall>
+      <cma_stall>0</cma_stall>
+      <cp>0.7 0.20 0</cp>
+      <area>0.10</area>
+      <air_density>1.2041</air_density>
+      <forward>0 -1 0</forward>
+      <upward>0 0 1</upward>
+      <link_name>${namespace}/zephyr_delta_wing/base_link</link_name>
+      <control_joint_name>
+        ${namespace}/zephyr_delta_wing/flap_left_joint
+      </control_joint_name>
+      <control_joint_rad_to_cl>-5.0</control_joint_rad_to_cl>
+  </plugin>
+  <plugin name="right_wing" filename="libLiftDragPlugin.so">
+      <a0>0.15</a0>
+      <cla>6.8</cla>
+      <cda>0.06417112299</cda>
+      <cma>-1.8</cma>
+      <alpha_stall>0.6391428111</alpha_stall>
+      <cla_stall>-3.85</cla_stall>
+      <cda_stall>-0.9233984055</cda_stall>
+      <cma_stall>0</cma_stall>
+      <cp>-0.7 0.20 0</cp>
+      <area>0.10</area>
+      <air_density>1.2041</air_density>
+      <forward>0 -1 0</forward>
+      <upward>0 0 1</upward>
+      <link_name>${namespace}/zephyr_delta_wing/base_link</link_name>
+      <control_joint_name>
+        ${namespace}/zephyr_delta_wing/flap_right_joint
+      </control_joint_name>
+      <control_joint_rad_to_cl>-5.0</control_joint_rad_to_cl>
+  </plugin>
+  <plugin name="left_rudder" filename="libLiftDragPlugin.so">
+      <a0>0.0</a0>
+      <cla>4.752798721</cla>
+      <cda>0.6417112299</cda>
+      <cma>-1.8</cma>
+      <alpha_stall>0.3391428111</alpha_stall>
+      <cla_stall>-3.85</cla_stall>
+      <cda_stall>-0.9233984055</cda_stall>
+      <cma_stall>0</cma_stall>
+      <cp>-0.76 0.30 0.025</cp>
+      <area>0.12</area>
+      <air_density>1.2041</air_density>
+      <forward>0 -1 0</forward>
+      <upward>1 0 0</upward>
+      <link_name>${namespace}/zephyr_delta_wing/base_link</link_name>
+  </plugin>
+  <plugin name="right_rudder" filename="libLiftDragPlugin.so">
+      <a0>0.0</a0>
+      <cla>4.752798721</cla>
+      <cda>0.6417112299</cda>
+      <cma>-1.8</cma>
+      <alpha_stall>0.3391428111</alpha_stall>
+      <cla_stall>-3.85</cla_stall>
+      <cda_stall>-0.9233984055</cda_stall>
+      <cma_stall>0</cma_stall>
+      <cp>0.76 0.30 0.025</cp>
+      <area>0.12</area>
+      <air_density>1.2041</air_density>
+      <forward>0 -1 0</forward>
+      <upward>1 0 0</upward>
+      <link_name>${namespace}/zephyr_delta_wing/base_link</link_name>
+  </plugin>
+  <plugin name="propeller_blade_1" filename="libLiftDragPlugin.so">
+      <a0>0.30</a0>
+      <alpha_stall>1.4</alpha_stall>
+      <cla>4.2500</cla>
+      <cda>0.10</cda>
+      <cma>0.00</cma>
+      <cla_stall>-0.025</cla_stall>
+      <cda_stall>0.0</cda_stall>
+      <cma_stall>0.0</cma_stall>
+      <area>0.02</area>
+      <air_density>1.2041</air_density>
+      <cp>0 0 0.074205</cp>
+      <forward>-1 0 0</forward>
+      <upward>0 -1 0</upward>
+      <link_name>${namespace}/zephyr_delta_wing/propeller</link_name>
+  </plugin>
+  <plugin name="propeller_blade_2" filename="libLiftDragPlugin.so">
+      <a0>0.30</a0>
+      <alpha_stall>1.4</alpha_stall>
+      <cla>4.2500</cla>
+      <cda>0.10</cda>
+      <cma>0.00</cma>
+      <cla_stall>-0.025</cla_stall>
+      <cda_stall>0.0</cda_stall>
+      <cma_stall>0.0</cma_stall>
+      <area>0.02</area>
+      <air_density>1.2041</air_density>
+      <cp>0 0 -0.074205</cp>
+      <forward>1 0 0</forward>
+      <upward>0 -1 0</upward>
+      <link_name>${namespace}/zephyr_delta_wing/propeller</link_name>
+  </plugin>
+  <plugin name="ardupilot_plugin" filename="libArduPilotPlugin.so">
+      <fdm_addr>127.0.0.1</fdm_addr>
+      <fdm_port_in>9002</fdm_port_in>
+      <fdm_port_out>9003</fdm_port_out>
+      <modelXYZToAirplaneXForwardZDown>0 0 0 3.141593 0 0</modelXYZToAirplaneXForwardZDown>
+      <gazeboXYZToNED>0 0 0 3.141593 0 0</gazeboXYZToNED>
+      <imuName>${namespace}/zephyr_delta_wing/zephyr/imu_link::imu_sensor</imuName>
+      <connectionTimeoutMaxCount>5</connectionTimeoutMaxCount>
+      <control channel="2">
+        <!--
+          incoming control command [0, 1]
+          so offset it by 0 to get [0, 1]
+          and divide max target by 1.
+            offset = 0
+            multiplier = 838 max rpm / 1 = 838
+        -->
+        <multiplier>838</multiplier>
+        <offset>0.0</offset>
+        <type>VELOCITY</type>
+        <p_gain>0.5</p_gain>
+        <i_gain>0</i_gain>
+        <d_gain>0</d_gain>
+        <i_max>0</i_max>
+        <i_min>0</i_min>
+        <cmd_max>2.0</cmd_max>
+        <cmd_min>0.0</cmd_min>
+        <jointName>${namespace}/zephyr_delta_wing/propeller_joint</jointName>
+      </control>
+      <control channel="1">
+        <multiplier>-1</multiplier>
+        <offset>-0.5</offset>
+        <type>POSITION</type>
+        <p_gain>10.0</p_gain>
+        <i_gain>0</i_gain>
+        <d_gain>0</d_gain>
+        <i_max>0</i_max>
+        <i_min>0</i_min>
+        <cmd_max>2.0</cmd_max>
+        <cmd_min>-2.0</cmd_min>
+        <jointName>${namespace}/zephyr_delta_wing/flap_right_joint</jointName>
+      </control>
+      <control channel="0">
+        <multiplier>-1</multiplier>
+        <offset>-0.5</offset>
+        <type>POSITION</type>
+        <p_gain>10.0</p_gain>
+        <i_gain>0</i_gain>
+        <d_gain>0</d_gain>
+        <i_max>0</i_max>
+        <i_min>0</i_min>
+        <cmd_max>2.0</cmd_max>
+        <cmd_min>-2.0</cmd_min>
+        <jointName>${namespace}/zephyr_delta_wing/flap_left_joint</jointName>
+      </control>
+  </plugin>
+  </gazebo>
 </robot>
