Commit message: [hawk] Fix typos

File: models/hawk/urdf/hawk.urdf.xacro (robot description, xacro)
@@ -39,5 +39,5 @@
   </xacro:property>
   <!-- Instantiate kopterworx mechanics "mechanics" -->
-  <xacro:include filename="$(find ardupilot_gazebo)/models/kopterworx/urdf/kopterworx_base.urdf.xacro" />
+  <xacro:include filename="$(find ardupilot_gazebo)/models/hawk/urdf/hawk_base.urdf.xacro" />
   <xacro:include filename="$(find rotors_description)/urdf/component_snippets.xacro" />
   <!-- Ardupilot plugin
@@ -117,7 +117,7 @@
     measurement_delay="0"
     unknown_delay="0.0"
-    noise_normal_position="0.0 0.0 0.0"
+    noise_normal_position="0.02 0.02 0.02"
     noise_normal_quaternion="0.0 0.0 0.0"
-    noise_normal_linear_velocity="0.0 0.0 0.0"
+    noise_normal_linear_velocity="0.05 0.05 0.05"
     noise_normal_angular_velocity="0.0 0.0 0.0"
     noise_uniform_position="0.0 0.0 0.0"

File: models/hawk/urdf/hawk_base.urdf.xacro (robot description, xacro)
@@ -6,5 +6,5 @@
   <!-- Body Properties -->
   <xacro:property name="rotor_velocity_slowdown_sim" value="15" />
-  <xacro:property name="mesh_file" value="ardupilot_gazebo/kopterworx/hawk/meshes/kopterworx_model_simple.dae" />
+  <xacro:property name="mesh_file" value="ardupilot_gazebo/models/kopterworx/meshes/kopterworx_model_simple.dae" />
   <xacro:property name="mesh_scale" value="0.075" />
   <xacro:property name="prop_scale" value="0.0015" />
